File: projects/ZZ-Servomotor/KiCad/pic16F628A.kicad_sch (KiCad schematic)
At the start: 2 parts, among them M1 Motor_Servo, U1 PIC16F628A-IP

Commit message: Documentation
Parts:
- added C1: 10uF, symbol Device:C_Polarized
- added R1: 12K, symbol Device:R_US
Connections:
- net +5V: now also C1.1, R1.2
- net GND: now also C1.2
- net at U1.4 (~{MCLR}/Vpp/RA5): now also R1.1
Changed lines of the file:
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@@
     (company "Ricardo Lima Caratti")
   )
-  (junction (at 69.85 31.75) (diameter 0) (color 0 0 0 0)
+  (junction (at 53.34 29.21) (diameter 0) (color 0 0 0 0)
+  )
+  (junction (at 113.03 31.75) (diameter 0) (color 0 0 0 0)
+  )
+  (junction (at 96.52 29.21) (diameter 0) (color 0 0 0 0)
+  )
+  (wire (pts (xy 113.03 77.47) (xy 113.03 83.82))
+    (stroke (width 0) (type default))
+  )
+  (wire (pts (xy 160.02 62.23) (xy 160.02 31.75))
+    (stroke (width 0) (type default))
   )
   (wire (pts (xy 50.8 53.34) (xy 69.85 53.34))
     (stroke (width 0) (type default))
   )
-  (wire (pts (xy 113.03 85.09) (xy 110.49 85.09))
-    (stroke (width 0) (type default))
-  )
-  (wire (pts (xy 113.03 77.47) (xy 113.03 85.09))
-    (stroke (width 0) (type default))
-  )
-  (wire (pts (xy 69.85 22.86) (xy 69.85 31.75))
-    (stroke (width 0) (type default))
-  )
-  (wire (pts (xy 69.85 55.88) (xy 69.85 57.15))
-    (stroke (width 0) (type default))
-  )
-  (wire (pts (xy 110.49 85.09) (xy 110.49 127))
-    (stroke (width 0) (type default))
-  )
-  (wire (pts (xy 50.8 55.88) (xy 69.85 55.88))
+  (wire (pts (xy 101.6 31.75) (xy 96.52 31.75))
+    (stroke (width 0) (type default))
+  )
+  (wire (pts (xy 109.22 31.75) (xy 113.03 31.75))
+    (stroke (width 0) (type default))
+  )
+  (wire (pts (xy 160.02 31.75) (xy 113.03 31.75))
+    (stroke (width 0) (type default))
+  )
+  (wire (pts (xy 53.34 29.21) (xy 96.52 29.21))
+    (stroke (width 0) (type default))
+  )
+  (wire (pts (xy 140.97 62.23) (xy 152.4 62.23))
     (stroke (width 0) (type default))
   )
@@
     (stroke (width 0) (type default))
   )
-  (wire (pts (xy 69.85 57.15) (xy 85.09 57.15))
+  (wire (pts (xy 53.34 29.21) (xy 53.34 50.8))
+    (stroke (width 0) (type default))
+  )
+  (wire (pts (xy 50.8 55.88) (xy 50.8 57.15))
+    (stroke (width 0) (type default))
+  )
+  (wire (pts (xy 96.52 29.21) (xy 96.52 31.75))
     (stroke (width 0) (type default))
   )
@@
     (stroke (width 0) (type default))
   )
-  (wire (pts (xy 113.03 31.75) (xy 69.85 31.75))
-    (stroke (width 0) (type default))
-  )
-  (wire (pts (xy 69.85 31.75) (xy 69.85 53.34))
-    (stroke (width 0) (type default))
-  )
-  (wire (pts (xy 53.34 50.8) (xy 53.34 35.56))
-    (stroke (width 0) (type default))
-  )
-  (symbol (lib_id "power:GND") (at 110.49 127 0) (unit 1)
-    (in_bom yes) (on_board yes) (dnp no) (fields_autoplaced)
-    (property "Reference" "#PWR03" (at 110.49 133.35 0)
-      (effects (font (size 1.27 1.27)) hide)
-    )
-    (property "Value" "GND" (at 110.49 132.08 0)
-      (effects (font (size 1.27 1.27)))
-    )
-    (property "Footprint" "" (at 110.49 127 0)
-      (effects (font (size 1.27 1.27)) hide)
-    )
-    (property "Datasheet" "" (at 110.49 127 0)
+  (wire (pts (xy 50.8 57.15) (xy 85.09 57.15))
+    (stroke (width 0) (type default))
+  )
+  (wire (pts (xy 69.85 48.26) (xy 69.85 53.34))
+    (stroke (width 0) (type default))
+  )
+  (symbol (lib_id "Device:R_US") (at 156.21 62.23 90) (unit 1)
+    (in_bom yes) (on_board yes) (dnp no) (fields_autoplaced)
+    (property "Reference" "R1" (at 156.21 55.88 90)
+      (effects (font (size 1.27 1.27)))
+    )
+    (property "Value" "12K" (at 156.21 58.42 90)
+      (effects (font (size 1.27 1.27)))
+    )
+    (property "Footprint" "" (at 156.464 61.214 90)
+      (effects (font (size 1.27 1.27)) hide)
+    )
+    (property "Datasheet" "~" (at 156.21 62.23 0)
+      (effects (font (size 1.27 1.27)) hide)
+    )
+    (pin "1")
+    (pin "2")
+    (instances
+      (project "Servo1"
+        (path "/73c37809-7617-4b9f-a70a-5c31575fa255"
+          (reference "R1") (unit 1)
+        )
+      )
+    )
+  )
+  (symbol (lib_id "Device:C_Polarized") (at 105.41 31.75 270) (unit 1)
+    (in_bom yes) (on_board yes) (dnp no) (fields_autoplaced)
+    (property "Reference" "C1" (at 106.299 24.13 90)
+      (effects (font (size 1.27 1.27)))
+    )
+    (property "Value" "10uF" (at 106.299 26.67 90)
+      (effects (font (size 1.27 1.27)))
+    )
+    (property "Footprint" "" (at 101.6 32.7152 0)
+      (effects (font (size 1.27 1.27)) hide)
+    )
+    (property "Datasheet" "~" (at 105.41 31.75 0)
+      (effects (font (size 1.27 1.27)) hide)
+    )
+    (pin "2")
+    (pin "1")
+    (instances
+      (project "Servo1"
+        (path "/73c37809-7617-4b9f-a70a-5c31575fa255"
+          (reference "C1") (unit 1)
+        )
+      )
+    )
+  )
+  (symbol (lib_id "power:GND") (at 113.03 83.82 0) (unit 1)
+    (in_bom yes) (on_board yes) (dnp no)
+    (property "Reference" "#PWR03" (at 113.03 90.17 0)
+      (effects (font (size 1.27 1.27)) hide)
+    )
+    (property "Value" "GND" (at 113.03 88.9 0)
+      (effects (font (size 1.27 1.27)))
+    )
+    (property "Footprint" "" (at 113.03 83.82 0)
+      (effects (font (size 1.27 1.27)) hide)
+    )
+    (property "Datasheet" "" (at 113.03 83.82 0)
       (effects (font (size 1.27 1.27)) hide)
     )
@@
     )
   )
-  (symbol (lib_id "power:GND") (at 53.34 35.56 180) (unit 1)
-    (in_bom yes) (on_board yes) (dnp no) (fields_autoplaced)
-    (property "Reference" "#PWR02" (at 53.34 29.21 0)
-      (effects (font (size 1.27 1.27)) hide)
-    )
-    (property "Value" "GND" (at 53.34 30.48 0)
-      (effects (font (size 1.27 1.27)))
-    )
-    (property "Footprint" "" (at 53.34 35.56 0)
-      (effects (font (size 1.27 1.27)) hide)
-    )
-    (property "Datasheet" "" (at 53.34 35.56 0)
+  (symbol (lib_id "power:GND") (at 53.34 29.21 180) (unit 1)
+    (in_bom yes) (on_board yes) (dnp no) (fields_autoplaced)
+    (property "Reference" "#PWR02" (at 53.34 22.86 0)
+      (effects (font (size 1.27 1.27)) hide)
+    )
+    (property "Value" "GND" (at 53.34 24.13 0)
+      (effects (font (size 1.27 1.27)))
+    )
+    (property "Footprint" "" (at 53.34 29.21 0)
+      (effects (font (size 1.27 1.27)) hide)
+    )
+    (property "Datasheet" "" (at 53.34 29.21 0)
       (effects (font (size 1.27 1.27)) hide)
     )
@@
         (path "/73c37809-7617-4b9f-a70a-5c31575fa255"
           (reference "#PWR02") (unit 1)
+        )
+      )
+    )
+  )
+  (symbol (lib_id "power:GND") (at 96.52 29.21 180) (unit 1)
+    (in_bom yes) (on_board yes) (dnp no) (fields_autoplaced)
+    (property "Reference" "#PWR04" (at 96.52 22.86 0)
+      (effects (font (size 1.27 1.27)) hide)
+    )
+    (property "Value" "GND" (at 96.52 24.13 0)
+      (effects (font (size 1.27 1.27)))
+    )
+    (property "Footprint" "" (at 96.52 29.21 0)
+      (effects (font (size 1.27 1.27)) hide)
+    )
+    (property "Datasheet" "" (at 96.52 29.21 0)
+      (effects (font (size 1.27 1.27)) hide)
+    )
+    (pin "1")
+    (instances
+      (project "Servo1"
+        (path "/73c37809-7617-4b9f-a70a-5c31575fa255"
+          (reference "#PWR04") (unit 1)
+        )
+      )
+    )
+  )
+  (symbol (lib_id "power:+5V") (at 113.03 31.75 0) (unit 1)
+    (in_bom yes) (on_board yes) (dnp no)
+    (property "Reference" "#PWR01" (at 113.03 24.13 0)
+      (effects (font (size 1.27 1.27)))
+    )
+    (property "Value" "+5V" (at 113.03 26.67 0)
+      (effects (font (size 1.27 1.27)))
+    )
+    (property "Footprint" "" (at 113.03 31.75 0)
+      (effects (font (size 1.27 1.27)) hide)
+    )
+    (property "Datasheet" "" (at 113.03 31.75 0)
+      (effects (font (size 1.27 1.27)) hide)
+    )
+    (pin "1")
+    (instances
+      (project "Servo1"
+        (path "/73c37809-7617-4b9f-a70a-5c31575fa255"
+          (reference "#PWR01") (unit 1)
         )
       )
@@
     )
   )
-  (symbol (lib_id "power:+5V") (at 69.85 22.86 0) (unit 1)
-    (in_bom yes) (on_board yes) (dnp no) (fields_autoplaced)
-    (property "Reference" "#PWR01" (at 69.85 26.67 0)
-      (effects (font (size 1.27 1.27)) hide)
-    )
-    (property "Value" "+5V" (at 69.85 17.78 0)
-      (effects (font (size 1.27 1.27)))
-    )
-    (property "Footprint" "" (at 69.85 22.86 0)
-      (effects (font (size 1.27 1.27)) hide)
-    )
-    (property "Datasheet" "" (at 69.85 22.86 0)
-      (effects (font (size 1.27 1.27)) hide)
-    )
-    (pin "1")
-    (instances
-      (project "Servo1"
-        (path "/73c37809-7617-4b9f-a70a-5c31575fa255"
-          (reference "#PWR01") (unit 1)
-        )
-      )
+  (symbol (lib_id "power:+5V") (at 69.85 48.26 0) (unit 1)
+    (in_bom yes) (on_board yes) (dnp no)
+    (property "Reference" "#PWR02" (at 69.85 40.64 0)
+      (effects (font (size 1.27 1.27)))
+    )
+    (property "Value" "+5V" (at 69.85 43.18 0)
+      (effects (font (size 1.27 1.27)))
+    )
+    (property "Footprint" "" (at 69.85 48.26 0)
+      (effects (font (size 1.27 1.27)) hide)
+    )
+    (property "Datasheet" "" (at 69.85 48.26 0)
+      (effects (font (size 1.27 1.27)) hide)
+    )
+    (pin "1")
+    (instances
+      (project "Servo1"
+        (path "/73c37809-7617-4b9f-a70a-5c31575fa255"
+          (reference "#PWR02") (unit 1)
+        )
+      )
