File: projects/10-74HC595/KiCad/PIC10F200_2x74HC595_2wires_16LEDs.kicad_sch (KiCad schematic)
At the start: 21 parts, among them U1 PIC10F200-IP, U2 74HC595

Commit message: Doc
Parts:
- removed D9: LED, symbol Device:LED
- removed R9: 360, symbol Device:R
- added D10, D11, D12, D13, D14, D15, D16, D17: LED, symbol Device:LED
- added R11, R12, R13, R14, R15, R16, R17, R18: 360, symbol Device:R
- added U3: 74HC595, symbol 74xx:74HC595
Connections:
- net +5V: now also U3.10 (~{SRCLR}), U3.16 (VCC)
- net GND: now also D10.1 (K), D11.1 (K), D12.1 (K), D13.1 (K), D14.1 (K), D15.1 (K), D16.1 (K), D17.1 (K), U3.13 (~{OE}), U3.8 (GND)
- net at U1.4 (GP1), U2.11 (SRCLK), U2.12 (RCLK): now also U3.11 (SRCLK), U3.12 (RCLK)
- net at U2.9 (QH'): now also U3.14 (SER)
- new net: R12.2, U3.1 (QB)
- new net: R11.2, U3.15 (QA)
- new net: R13.2, U3.2 (QC)
- new net: R14.2, U3.3 (QD)
- new net: R15.2, U3.4 (QE)
- new net: R16.2, U3.5 (QF)
- new net: R17.2, U3.6 (QG)
- new net: R18.2, U3.7 (QH)
- new net: D12.2 (A), R13.1
- new net: D15.2 (A), R16.1
- new net: D10.2 (A), R11.1
- new net: D11.2 (A), R12.1
- new net: D17.2 (A), R18.1
- new net: D16.2 (A), R17.1
- new net: D13.2 (A), R14.1
- new net: D14.2 (A), R15.1
Other:
- title: PIC10F200 and 74HC595 two wires setup -> PIC10F200 and 2 x74HC595 with  two wires interface setup
- moved on the sheet: D2, D3, D4, D5, D6, D7, D8, R2, R3, R4, R5, R6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
