File: projects/10-74HC595/KiCad/PIC10F200_74HC595_2wires_8LEDs.kicad_sch (KiCad schematic)
At the start: 21 parts, among them U1 PIC10F200-IP, U2 74HC595

Commit message: Doc
Parts:
- removed D9: LED, symbol Device:LED
- removed R9: 360, symbol Device:R
Changed lines of the file:
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@@
     (company "Ricardo Lima Caratti")
   )
-  (junction (at 60.96 113.03) (diameter 0) (color 0 0 0 0)
-  )
   (junction (at 123.19 88.9) (diameter 0) (color 0 0 0 0)
   )
@@
     (stroke (width 0) (type default))
   )
-  (wire (pts (xy 68.58 128.27) (xy 77.47 128.27))
-    (stroke (width 0) (type default))
-  )
   (wire (pts (xy 123.19 88.9) (xy 123.19 92.71))
     (stroke (width 0) (type default))
@@
     (stroke (width 0) (type default))
   )
-  (wire (pts (xy 113.03 82.55) (xy 113.03 128.27))
-    (stroke (width 0) (type default))
-  )
   (wire (pts (xy 104.14 62.23) (xy 104.14 33.02))
     (stroke (width 0) (type default))
@@
     (stroke (width 0) (type default))
   )
-  (wire (pts (xy 85.09 128.27) (xy 113.03 128.27))
-    (stroke (width 0) (type default))
-  )
   (wire (pts (xy 113.03 64.77) (xy 101.6 64.77))
     (stroke (width 0) (type default))
@@
   )
   (wire (pts (xy 142.24 53.34) (xy 179.07 53.34))
-    (stroke (width 0) (type default))
-  )
-  (wire (pts (xy 60.96 113.03) (xy 60.96 128.27))
     (stroke (width 0) (type default))
   )
@@
     )
   )
-  (symbol (lib_id "Device:LED") (at 64.77 128.27 0) (unit 1)
-    (in_bom yes) (on_board yes) (dnp no)
-    (property "Reference" "D9" (at 63.1825 121.92 0)
-      (effects (font (size 1.27 1.27)))
-    )
-    (property "Value" "LED" (at 63.1825 124.46 0)
-      (effects (font (size 1.27 1.27)))
-    )
-    (property "Footprint" "" (at 64.77 128.27 0)
-      (effects (font (size 1.27 1.27)) hide)
-    )
-    (property "Datasheet" "~" (at 64.77 128.27 0)
-      (effects (font (size 1.27 1.27)) hide)
-    )
-    (pin "1")
-    (pin "2")
-    (instances
-      (project "PIC10F200_74HC595_2wires_8LEDs"
-        (path "/25a1316a-e1e9-47cf-8bb8-a0bf08fb5198"
-          (reference "D9") (unit 1)
-        )
-      )
-    )
-  )
   (symbol (lib_id "Device:R") (at 81.28 46.99 90) (unit 1)
     (in_bom yes) (on_board yes) (dnp no) (fields_autoplaced)
@@
         )
       )
-    )
-  )
-  (symbol (lib_id "Device:R") (at 81.28 128.27 90) (unit 1)
-    (in_bom yes) (on_board yes) (dnp no)
-    (property "Reference" "R9" (at 81.28 121.92 90)
-      (effects (font (size 1.27 1.27)))
-    )
-    (property "Value" "360" (at 81.28 124.46 90)
-      (effects (font (size 1.27 1.27)))
-    )
-    (property "Footprint" "" (at 81.28 130.048 90)
-      (effects (font (size 1.27 1.27)) hide)
-    )
-    (property "Datasheet" "~" (at 81.28 128.27 0)
-      (effects (font (size 1.27 1.27)) hide)
-    )
-    (pin "1")
-    (pin "2")
-    (instances
-      (project "PIC10F200_74HC595_2wires_8LEDs"
-        (path "/25a1316a-e1e9-47cf-8bb8-a0bf08fb5198"
-          (reference "R9") (unit 1)
-        )
-      )
