File: projects/10-74HC595/KiCad/PIC10F200_2x74HC595_3wires_16LEDs.kicad_sch (KiCad schematic)
At the start: 36 parts, among them U1 PIC10F200-IP, U2 74HC595, U3 74HC595

Commit message: Doc
Other:
- title: PIC10F200 and 2 x74HC595 with  two wires interface setup -> PIC10F200 and 2 x74HC595 with three wires interface setup
Changed lines of the file:
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@@
   (paper "User" 299.999 240.995)
   (title_block
-    (title "PIC10F200 and 2 x74HC595 with  two wires interface setup")
+    (title "PIC10F200 and 2 x74HC595 with three wires interface setup")
     (company "Ricardo Lima Caratti")
   )
