File: projects/01-Blink/Kicad/PIC16F628A_blink.kicad_sch (KiCad schematic)
At the start: 6 parts, among them U1 PIC16F628A-IP

Commit message: Doc
Parts:
- removed C1: 10uF, symbol Device:C_Polarized
- removed C2: 100nF, symbol Device:C
- R1: value 12K -> 10K
Changed lines of the file:
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@@
     (comment 1 "A minimalist project to blink an LED using the PIC16F628A. ")
-  )
-  (junction (at 90.17 55.88) (diameter 0) (color 0 0 0 0)
   )
   (junction (at 90.17 101.6) (diameter 0) (color 0 0 0 0)
   )
-  (wire (pts (xy 90.17 55.88) (xy 96.52 55.88))
-    (stroke (width 0) (type default))
-  )
   (wire (pts (xy 29.21 73.66) (xy 33.02 73.66))
-    (stroke (width 0) (type default))
-  )
-  (wire (pts (xy 104.14 55.88) (xy 110.49 55.88))
     (stroke (width 0) (type default))
   )
@@
     (stroke (width 0) (type default))
   )
-  (wire (pts (xy 90.17 55.88) (xy 90.17 66.04))
+  (wire (pts (xy 90.17 53.34) (xy 90.17 66.04))
     (stroke (width 0) (type default))
   )
@@
     (stroke (width 0) (type default))
   )
-  (wire (pts (xy 67.31 55.88) (xy 73.66 55.88))
-    (stroke (width 0) (type default))
-  )
   (wire (pts (xy 21.59 73.66) (xy 19.05 73.66))
-    (stroke (width 0) (type default))
-  )
-  (wire (pts (xy 81.28 55.88) (xy 90.17 55.88))
     (stroke (width 0) (type default))
   )
@@
   )
   (wire (pts (xy 135.89 86.36) (xy 146.05 86.36))
-    (stroke (width 0) (type default))
-  )
-  (wire (pts (xy 90.17 53.34) (xy 90.17 55.88))
     (stroke (width 0) (type default))
   )
@@
       (effects (font (size 1.27 1.27)))
     )
-    (property "Value" "12K" (at 132.08 82.55 90)
+    (property "Value" "10K" (at 132.08 82.55 90)
       (effects (font (size 1.27 1.27)))
     )
@@
     )
   )
-  (symbol (lib_id "power:GND") (at 110.49 55.88 0) (unit 1)
-    (in_bom yes) (on_board yes) (dnp no) (fields_autoplaced)
-    (property "Reference" "#PWR03" (at 110.49 62.23 0)
-      (effects (font (size 1.27 1.27)) hide)
-    )
-    (property "Value" "GND" (at 110.49 60.96 0)
-      (effects (font (size 1.27 1.27)))
-    )
-    (property "Footprint" "" (at 110.49 55.88 0)
-      (effects (font (size 1.27 1.27)) hide)
-    )
-    (property "Datasheet" "" (at 110.49 55.88 0)
-      (effects (font (size 1.27 1.27)) hide)
-    )
-    (pin "1")
-    (instances
-      (project "PIC16F628A_blink"
-        (path "/e310d602-5c89-43bf-b83f-8bd293d0af3f"
-          (reference "#PWR03") (unit 1)
-        )
-      )
-    )
-  )
   (symbol (lib_id "power:GND") (at 19.05 73.66 0) (unit 1)
     (in_bom yes) (on_board yes) (dnp no) (fields_autoplaced)
@@
         (path "/e310d602-5c89-43bf-b83f-8bd293d0af3f"
           (reference "#PWR05") (unit 1)
-        )
-      )
-    )
-  )
-  (symbol (lib_id "Device:C_Polarized") (at 100.33 55.88 90) (unit 1)
-    (in_bom yes) (on_board yes) (dnp no) (fields_autoplaced)
-    (property "Reference" "C1" (at 99.441 48.26 90)
-      (effects (font (size 1.27 1.27)))
-    )
-    (property "Value" "10uF" (at 99.441 50.8 90)
-      (effects (font (size 1.27 1.27)))
-    )
-    (property "Footprint" "" (at 104.14 54.9148 0)
-      (effects (font (size 1.27 1.27)) hide)
-    )
-    (property "Datasheet" "~" (at 100.33 55.88 0)
-      (effects (font (size 1.27 1.27)) hide)
-    )
-    (pin "1")
-    (pin "2")
-    (instances
-      (project "PIC16F628A_blink"
-        (path "/e310d602-5c89-43bf-b83f-8bd293d0af3f"
-          (reference "C1") (unit 1)
-        )
-      )
-    )
-  )
-  (symbol (lib_id "power:GND") (at 67.31 55.88 0) (unit 1)
-    (in_bom yes) (on_board yes) (dnp no) (fields_autoplaced)
-    (property "Reference" "#PWR06" (at 67.31 62.23 0)
-      (effects (font (size 1.27 1.27)) hide)
-    )
-    (property "Value" "GND" (at 67.31 60.96 0)
-      (effects (font (size 1.27 1.27)))
-    )
-    (property "Footprint" "" (at 67.31 55.88 0)
-      (effects (font (size 1.27 1.27)) hide)
-    )
-    (property "Datasheet" "" (at 67.31 55.88 0)
-      (effects (font (size 1.27 1.27)) hide)
-    )
-    (pin "1")
-    (instances
-      (project "PIC16F628A_blink"
-        (path "/e310d602-5c89-43bf-b83f-8bd293d0af3f"
-          (reference "#PWR06") (unit 1)
         )
       )
@@
         )
       )
-    )
-  )
-  (symbol (lib_id "Device:C") (at 77.47 55.88 90) (unit 1)
-    (in_bom yes) (on_board yes) (dnp no) (fields_autoplaced)
-    (property "Reference" "C2" (at 77.47 48.26 90)
-      (effects (font (size 1.27 1.27)))
-    )
-    (property "Value" "100nF" (at 77.47 50.8 90)
-      (effects (font (size 1.27 1.27)))
-    )
-    (property "Footprint" "" (at 81.28 54.9148 0)
-      (effects (font (size 1.27 1.27)) hide)
-    )
-    (property "Datasheet" "~" (at 77.47 55.88 0)
-      (effects (font (size 1.27 1.27)) hide)
-    )
-    (pin "1")
-    (pin "2")
-    (instances
-      (project "PIC16F628A_blink"
-        (path "/e310d602-5c89-43bf-b83f-8bd293d0af3f"
-          (reference "C2") (unit 1)
-        )
-      )
