File: projects/02-LED_CONTROL/Kicad/PIC12F675_blink3LEds.kicad_sch (KiCad schematic)
At the start: 10 parts, among them U1 PIC12F675-IP

Commit message: Doc
Parts:
- removed C1: 10uF, symbol Device:C_Polarized
- removed C2: 100nF, symbol Device:C
- R1: value 12K -> 10K
Other:
- title: PIC16F628A for Beginners - 1 -> PIC16F675 for Beginners - 1
- moved on the sheet: R1
Changed lines of the file:
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@@
   (paper "User" 203.2 177.8)
   (title_block
-    (title "PIC16F628A for Beginners - 1")
+    (title "PIC16F675 for Beginners - 1")
     (company "Ricardo Lima Caratti")
     (comment 1 "Controlling three LEDs using PIC12F675. ")
   )
-  (junction (at 90.17 55.88) (diameter 0) (color 0 0 0 0)
-  )
   (junction (at 39.37 81.28) (diameter 0) (color 0 0 0 0)
   )
-  (wire (pts (xy 90.17 55.88) (xy 96.52 55.88))
-    (stroke (width 0) (type default))
-  )
   (wire (pts (xy 49.53 69.85) (xy 53.34 69.85))
     (stroke (width 0) (type default))
@@
     (stroke (width 0) (type default))
   )
-  (wire (pts (xy 104.14 55.88) (xy 110.49 55.88))
-    (stroke (width 0) (type default))
-  )
   (wire (pts (xy 30.48 81.28) (xy 39.37 81.28))
     (stroke (width 0) (type default))
@@
     (stroke (width 0) (type default))
   )
-  (wire (pts (xy 105.41 78.74) (xy 127 78.74))
+  (wire (pts (xy 105.41 78.74) (xy 114.3 78.74))
     (stroke (width 0) (type default))
   )
@@
     (stroke (width 0) (type default))
   )
-  (wire (pts (xy 90.17 55.88) (xy 90.17 66.04))
-    (stroke (width 0) (type default))
-  )
-  (wire (pts (xy 67.31 55.88) (xy 73.66 55.88))
+  (wire (pts (xy 90.17 53.34) (xy 90.17 66.04))
     (stroke (width 0) (type default))
   )
@@
     (stroke (width 0) (type default))
   )
-  (wire (pts (xy 81.28 55.88) (xy 90.17 55.88))
-    (stroke (width 0) (type default))
-  )
   (wire (pts (xy 30.48 83.82) (xy 30.48 81.28))
     (stroke (width 0) (type default))
@@
     (stroke (width 0) (type default))
   )
-  (wire (pts (xy 134.62 78.74) (xy 144.78 78.74))
-    (stroke (width 0) (type default))
-  )
-  (wire (pts (xy 90.17 53.34) (xy 90.17 55.88))
+  (wire (pts (xy 121.92 78.74) (xy 132.08 78.74))
     (stroke (width 0) (type default))
   )
@@
     )
   )
-  (symbol (lib_id "Device:R") (at 130.81 78.74 90) (unit 1)
-    (in_bom yes) (on_board yes) (dnp no) (fields_autoplaced)
-    (property "Reference" "R1" (at 130.81 72.39 90)
-      (effects (font (size 1.27 1.27)))
-    )
-    (property "Value" "12K" (at 130.81 74.93 90)
-      (effects (font (size 1.27 1.27)))
-    )
-    (property "Footprint" "" (at 130.81 80.518 90)
-      (effects (font (size 1.27 1.27)) hide)
-    )
-    (property "Datasheet" "~" (at 130.81 78.74 0)
+  (symbol (lib_id "Device:R") (at 118.11 78.74 90) (unit 1)
+    (in_bom yes) (on_board yes) (dnp no) (fields_autoplaced)
+    (property "Reference" "R1" (at 118.11 72.39 90)
+      (effects (font (size 1.27 1.27)))
+    )
+    (property "Value" "10K" (at 118.11 74.93 90)
+      (effects (font (size 1.27 1.27)))
+    )
+    (property "Footprint" "" (at 118.11 80.518 90)
+      (effects (font (size 1.27 1.27)) hide)
+    )
+    (property "Datasheet" "~" (at 118.11 78.74 0)
       (effects (font (size 1.27 1.27)) hide)
     )
@@
     )
   )
-  (symbol (lib_id "power:+5V") (at 144.78 78.74 0) (unit 1)
-    (in_bom yes) (on_board yes) (dnp no) (fields_autoplaced)
-    (property "Reference" "#PWR04" (at 144.78 82.55 0)
-      (effects (font (size 1.27 1.27)) hide)
-    )
-    (property "Value" "+5V" (at 144.78 73.66 0)
-      (effects (font (size 1.27 1.27)))
-    )
-    (property "Footprint" "" (at 144.78 78.74 0)
-      (effects (font (size 1.27 1.27)) hide)
-    )
-    (property "Datasheet" "" (at 144.78 78.74 0)
+  (symbol (lib_id "power:+5V") (at 132.08 78.74 0) (unit 1)
+    (in_bom yes) (on_board yes) (dnp no) (fields_autoplaced)
+    (property "Reference" "#PWR04" (at 132.08 82.55 0)
+      (effects (font (size 1.27 1.27)) hide)
+    )
+    (property "Value" "+5V" (at 132.08 73.66 0)
+      (effects (font (size 1.27 1.27)))
+    )
+    (property "Footprint" "" (at 132.08 78.74 0)
+      (effects (font (size 1.27 1.27)) hide)
+    )
+    (property "Datasheet" "" (at 132.08 78.74 0)
       (effects (font (size 1.27 1.27)) hide)
     )
@@
     )
   )
-  (symbol (lib_id "power:GND") (at 110.49 55.88 0) (unit 1)
-    (in_bom yes) (on_board yes) (dnp no) (fields_autoplaced)
-    (property "Reference" "#PWR03" (at 110.49 62.23 0)
-      (effects (font (size 1.27 1.27)) hide)
-    )
-    (property "Value" "GND" (at 110.49 60.96 0)
-      (effects (font (size 1.27 1.27)))
-    )
-    (property "Footprint" "" (at 110.49 55.88 0)
-      (effects (font (size 1.27 1.27)) hide)
-    )
-    (property "Datasheet" "" (at 110.49 55.88 0)
-      (effects (font (size 1.27 1.27)) hide)
-    )
-    (pin "1")
-    (instances
-      (project "PIC12F675_blink3LEds"
-        (path "/e310d602-5c89-43bf-b83f-8bd293d0af3f"
-          (reference "#PWR03") (unit 1)
-        )
-      )
-    )
-  )
-  (symbol (lib_id "Device:C_Polarized") (at 100.33 55.88 90) (unit 1)
-    (in_bom yes) (on_board yes) (dnp no) (fields_autoplaced)
-    (property "Reference" "C1" (at 99.441 48.26 90)
-      (effects (font (size 1.27 1.27)))
-    )
-    (property "Value" "10uF" (at 99.441 50.8 90)
-      (effects (font (size 1.27 1.27)))
-    )
-    (property "Footprint" "" (at 104.14 54.9148 0)
-      (effects (font (size 1.27 1.27)) hide)
-    )
-    (property "Datasheet" "~" (at 100.33 55.88 0)
-      (effects (font (size 1.27 1.27)) hide)
-    )
-    (pin "1")
-    (pin "2")
-    (instances
-      (project "PIC12F675_blink3LEds"
-        (path "/e310d602-5c89-43bf-b83f-8bd293d0af3f"
-          (reference "C1") (unit 1)
-        )
-      )
-    )
-  )
-  (symbol (lib_id "power:GND") (at 67.31 55.88 0) (unit 1)
-    (in_bom yes) (on_board yes) (dnp no) (fields_autoplaced)
-    (property "Reference" "#PWR06" (at 67.31 62.23 0)
-      (effects (font (size 1.27 1.27)) hide)
-    )
-    (property "Value" "GND" (at 67.31 60.96 0)
-      (effects (font (size 1.27 1.27)))
-    )
-    (property "Footprint" "" (at 67.31 55.88 0)
-      (effects (font (size 1.27 1.27)) hide)
-    )
-    (property "Datasheet" "" (at 67.31 55.88 0)
-      (effects (font (size 1.27 1.27)) hide)
-    )
-    (pin "1")
-    (instances
-      (project "PIC12F675_blink3LEds"
-        (path "/e310d602-5c89-43bf-b83f-8bd293d0af3f"
-          (reference "#PWR06") (unit 1)
-        )
-      )
-    )
-  )
   (symbol (lib_id "Device:LED") (at 45.72 69.85 0) (unit 1)
     (in_bom yes) (on_board yes) (dnp no) (fields_autoplaced)
@@
         )
       )
-    )
-  )
-  (symbol (lib_id "Device:C") (at 77.47 55.88 90) (unit 1)
-    (in_bom yes) (on_board yes) (dnp no) (fields_autoplaced)
-    (property "Reference" "C2" (at 77.47 48.26 90)
-      (effects (font (size 1.27 1.27)))
-    )
-    (property "Value" "100nF" (at 77.47 50.8 90)
-      (effects (font (size 1.27 1.27)))
-    )
-    (property "Footprint" "" (at 81.28 54.9148 0)
-      (effects (font (size 1.27 1.27)) hide)
-    )
-    (property "Datasheet" "~" (at 77.47 55.88 0)
-      (effects (font (size 1.27 1.27)) hide)
-    )
-    (pin "1")
-    (pin "2")
-    (instances
-      (project "PIC12F675_blink3LEds"
-        (path "/e310d602-5c89-43bf-b83f-8bd293d0af3f"
-          (reference "C2") (unit 1)
-        )
-      )
