File: projects/02-LED_CONTROL/Kicad/PIC16F628A_8_LEDs.kicad_sch (KiCad schematic)
At the start: 20 parts, among them U1 PIC16F628A-IP

Commit message: Doc
Parts:
- removed C1: 10uF, symbol Device:C_Polarized
- removed C2: 100nF, symbol Device:C
- R1: value 12K -> 10K
Other:
- moved on the sheet: D1, D2, D3, D4, D5, D6, D7, D8, R1, R2, R3, R4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
