File: projects/03-PIC16F_LCD16x2/KiCad/PIC16F628A_LCD16x2.kicad_sch (KiCad schematic)
At the start: 6 parts, among them U1 PIC16F628A-IP, U2 LCD-016N002L

Commit message: Documentation
Connections:
- net +5V: now also U2.A1
- net GND: now also U2.K1
Other:
- moved on the sheet: C1, C2, R1, RV1, U1, U2

Commit message: Doc
Parts:
- removed C1: 10uF, symbol Device:C_Polarized
- removed C2: 100nF, symbol Device:C
- R1: value 12K -> 10K
Changed lines of the file:
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@@
     (comment 1 "LCD 16x2 nd PIC16F628A")
   )
-  (junction (at 88.9 39.37) (diameter 0) (color 0 0 0 0)
-  )
   (junction (at 165.1 39.37) (diameter 0) (color 0 0 0 0)
   )
@@
     (stroke (width 0) (type default))
   )
-  (wire (pts (xy 88.9 39.37) (xy 82.55 39.37))
-    (stroke (width 0) (type default))
-  )
   (wire (pts (xy 116.84 62.23) (xy 140.97 62.23))
     (stroke (width 0) (type default))
@@
     (stroke (width 0) (type default))
   )
-  (wire (pts (xy 74.93 39.37) (xy 68.58 39.37))
-    (stroke (width 0) (type default))
-  )
   (wire (pts (xy 165.1 39.37) (xy 184.15 39.37))
     (stroke (width 0) (type default))
@@
     (stroke (width 0) (type default))
   )
-  (wire (pts (xy 88.9 39.37) (xy 88.9 49.53))
-    (stroke (width 0) (type default))
-  )
   (wire (pts (xy 200.66 80.01) (xy 184.15 80.01))
     (stroke (width 0) (type default))
@@
     (stroke (width 0) (type default))
   )
-  (wire (pts (xy 111.76 39.37) (xy 105.41 39.37))
-    (stroke (width 0) (type default))
-  )
   (wire (pts (xy 175.26 52.07) (xy 196.85 52.07))
     (stroke (width 0) (type default))
@@
     (stroke (width 0) (type default))
   )
-  (wire (pts (xy 97.79 39.37) (xy 88.9 39.37))
-    (stroke (width 0) (type default))
-  )
   (wire (pts (xy 116.84 64.77) (xy 138.43 64.77))
     (stroke (width 0) (type default))
@@
     (stroke (width 0) (type default))
   )
-  (wire (pts (xy 88.9 36.83) (xy 88.9 39.37))
+  (wire (pts (xy 88.9 36.83) (xy 88.9 49.53))
     (stroke (width 0) (type default))
   )
@@
       (effects (font (size 1.27 1.27)))
     )
-    (property "Value" "12K" (at 46.99 66.04 90)
+    (property "Value" "10K" (at 46.99 66.04 90)
       (effects (font (size 1.27 1.27)))
     )
@@
         (path "/e310d602-5c89-43bf-b83f-8bd293d0af3f"
           (reference "#PWR07") (unit 1)
-        )
-      )
-    )
-  )
-  (symbol (lib_id "power:GND") (at 68.58 39.37 0) (mirror y) (unit 1)
-    (in_bom yes) (on_board yes) (dnp no) (fields_autoplaced)
-    (property "Reference" "#PWR03" (at 68.58 45.72 0)
-      (effects (font (size 1.27 1.27)) hide)
-    )
-    (property "Value" "GND" (at 68.58 44.45 0)
-      (effects (font (size 1.27 1.27)))
-    )
-    (property "Footprint" "" (at 68.58 39.37 0)
-      (effects (font (size 1.27 1.27)) hide)
-    )
-    (property "Datasheet" "" (at 68.58 39.37 0)
-      (effects (font (size 1.27 1.27)) hide)
-    )
-    (pin "1")
-    (instances
-      (project "PIC16F628A_LCD16x2"
-        (path "/e310d602-5c89-43bf-b83f-8bd293d0af3f"
-          (reference "#PWR03") (unit 1)
-        )
-      )
-    )
-  )
-  (symbol (lib_id "Device:C_Polarized") (at 78.74 39.37 270) (mirror x) (unit 1)
-    (in_bom yes) (on_board yes) (dnp no) (fields_autoplaced)
-    (property "Reference" "C1" (at 79.629 31.75 90)
-      (effects (font (size 1.27 1.27)))
-    )
-    (property "Value" "10uF" (at 79.629 34.29 90)
-      (effects (font (size 1.27 1.27)))
-    )
-    (property "Footprint" "" (at 74.93 38.4048 0)
-      (effects (font (size 1.27 1.27)) hide)
-    )
-    (property "Datasheet" "~" (at 78.74 39.37 0)
-      (effects (font (size 1.27 1.27)) hide)
-    )
-    (pin "1")
-    (pin "2")
-    (instances
-      (project "PIC16F628A_LCD16x2"
-        (path "/e310d602-5c89-43bf-b83f-8bd293d0af3f"
-          (reference "C1") (unit 1)
-        )
-      )
-    )
-  )
-  (symbol (lib_id "power:GND") (at 111.76 39.37 0) (mirror y) (unit 1)
-    (in_bom yes) (on_board yes) (dnp no) (fields_autoplaced)
-    (property "Reference" "#PWR06" (at 111.76 45.72 0)
-      (effects (font (size 1.27 1.27)) hide)
-    )
-    (property "Value" "GND" (at 111.76 44.45 0)
-      (effects (font (size 1.27 1.27)))
-    )
-    (property "Footprint" "" (at 111.76 39.37 0)
-      (effects (font (size 1.27 1.27)) hide)
-    )
-    (property "Datasheet" "" (at 111.76 39.37 0)
-      (effects (font (size 1.27 1.27)) hide)
-    )
-    (pin "1")
-    (instances
-      (project "PIC16F628A_LCD16x2"
-        (path "/e310d602-5c89-43bf-b83f-8bd293d0af3f"
-          (reference "#PWR06") (unit 1)
         )
       )
@@
         )
       )
-    )
-  )
-  (symbol (lib_id "Device:C") (at 101.6 39.37 270) (mirror x) (unit 1)
-    (in_bom yes) (on_board yes) (dnp no) (fields_autoplaced)
-    (property "Reference" "C2" (at 101.6 31.75 90)
-      (effects (font (size 1.27 1.27)))
-    )
-    (property "Value" "100nF" (at 101.6 34.29 90)
-      (effects (font (size 1.27 1.27)))
-    )
-    (property "Footprint" "" (at 97.79 38.4048 0)
-      (effects (font (size 1.27 1.27)) hide)
-    )
-    (property "Datasheet" "~" (at 101.6 39.37 0)
-      (effects (font (size 1.27 1.27)) hide)
-    )
-    (pin "1")
-    (pin "2")
-    (instances
-      (project "PIC16F628A_LCD16x2"
-        (path "/e310d602-5c89-43bf-b83f-8bd293d0af3f"
-          (reference "C2") (unit 1)
-        )
-      )
