File: projects/03-PIC16F_LCD16x2/KiCad/pic16F876A_lcd16x2 copy.kicad_sch (KiCad schematic)
At the start: 8 parts, among them U1 PIC16F876-XXISO, U2 LCD-016N002L, Y1 8MHz

Commit message: Doc
Parts:
- removed C1: 10uF, symbol Device:C_Polarized
- R1: value 12K -> 10K
Changed lines of the file:
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@@
     (company "Ricardo Lima Caratti")
   )
-  (junction (at 82.55 40.64) (diameter 0) (color 0 0 0 0)
-  )
   (junction (at 110.49 87.63) (diameter 0) (color 0 0 0 0)
   )
@@
     (stroke (width 0) (type default))
   )
-  (wire (pts (xy 72.39 40.64) (xy 67.31 40.64))
-    (stroke (width 0) (type default))
-  )
   (wire (pts (xy 110.49 102.87) (xy 121.92 102.87))
     (stroke (width 0) (type default))
@@
     (stroke (width 0) (type default))
   )
-  (wire (pts (xy 80.01 40.64) (xy 82.55 40.64))
-    (stroke (width 0) (type default))
-  )
   (wire (pts (xy 102.87 73.66) (xy 102.87 81.28))
     (stroke (width 0) (type default))
@@
     (stroke (width 0) (type default))
   )
-  (wire (pts (xy 82.55 40.64) (xy 83.82 40.64))
-    (stroke (width 0) (type default))
-  )
   (wire (pts (xy 80.01 124.46) (xy 82.55 124.46))
     (stroke (width 0) (type default))
@@
     (stroke (width 0) (type default))
   )
-  (wire (pts (xy 67.31 38.1) (xy 67.31 40.64))
-    (stroke (width 0) (type default))
-  )
   (wire (pts (xy 102.87 63.5) (xy 102.87 66.04))
     (stroke (width 0) (type default))
@@
     (stroke (width 0) (type default))
   )
-  (wire (pts (xy 82.55 40.64) (xy 82.55 63.5))
+  (wire (pts (xy 82.55 57.15) (xy 82.55 63.5))
     (stroke (width 0) (type default))
   )
@@
       (effects (font (size 1.27 1.27)))
     )
-    (property "Value" "12K" (at 99.06 69.85 90)
+    (property "Value" "10K" (at 99.06 69.85 90)
       (effects (font (size 1.27 1.27)))
     )
@@
         (path "/73c37809-7617-4b9f-a70a-5c31575fa255"
           (reference "R1") (unit 1)
-        )
-      )
-    )
-  )
-  (symbol (lib_id "Device:C_Polarized") (at 76.2 40.64 270) (unit 1)
-    (in_bom yes) (on_board yes) (dnp no) (fields_autoplaced)
-    (property "Reference" "C1" (at 77.089 33.02 90)
-      (effects (font (size 1.27 1.27)))
-    )
-    (property "Value" "10uF" (at 77.089 35.56 90)
-      (effects (font (size 1.27 1.27)))
-    )
-    (property "Footprint" "" (at 72.39 41.6052 0)
-      (effects (font (size 1.27 1.27)) hide)
-    )
-    (property "Datasheet" "~" (at 76.2 40.64 0)
-      (effects (font (size 1.27 1.27)) hide)
-    )
-    (pin "1")
-    (pin "2")
-    (instances
-      (project "pic16F876A_lcd16x2 copy"
-        (path "/73c37809-7617-4b9f-a70a-5c31575fa255"
-          (reference "C1") (unit 1)
         )
       )
@@
     )
   )
-  (symbol (lib_id "power:GND") (at 67.31 38.1 180) (unit 1)
-    (in_bom yes) (on_board yes) (dnp no) (fields_autoplaced)
-    (property "Reference" "#PWR04" (at 67.31 31.75 0)
-      (effects (font (size 1.27 1.27)) hide)
-    )
-    (property "Value" "GND" (at 67.31 33.02 0)
-      (effects (font (size 1.27 1.27)))
-    )
-    (property "Footprint" "" (at 67.31 38.1 0)
-      (effects (font (size 1.27 1.27)) hide)
-    )
-    (property "Datasheet" "" (at 67.31 38.1 0)
-      (effects (font (size 1.27 1.27)) hide)
-    )
-    (pin "1")
-    (instances
-      (project "pic16F876A_lcd16x2 copy"
-        (path "/73c37809-7617-4b9f-a70a-5c31575fa255"
-          (reference "#PWR04") (unit 1)
-        )
-      )
-    )
-  )
   (symbol (lib_id "Device:Crystal") (at 110.49 91.44 270) (unit 1)
     (in_bom yes) (on_board yes) (dnp no) (fields_autoplaced)
@@
     )
   )
-  (symbol (lib_id "power:+5V") (at 83.82 40.64 0) (unit 1)
-    (in_bom yes) (on_board yes) (dnp no)
-    (property "Reference" "#PWR01" (at 83.82 33.02 0)
-      (effects (font (size 1.27 1.27)))
-    )
-    (property "Value" "+5V" (at 83.82 35.56 0)
-      (effects (font (size 1.27 1.27)))
-    )
-    (property "Footprint" "" (at 83.82 40.64 0)
-      (effects (font (size 1.27 1.27)) hide)
-    )
-    (property "Datasheet" "" (at 83.82 40.64 0)
-      (effects (font (size 1.27 1.27)) hide)
-    )
+  (symbol (lib_id "power:+5V") (at 82.55 57.15 0) (unit 1)
+    (in_bom yes) (on_board yes) (dnp no)
+    (property "Reference" "#PWR01" (at 82.55 49.53 0)
+      (effects (font (size 1.27 1.27)))
+    )
+    (property "Value" "+5V" (at 82.55 52.07 0)
+      (effects (font (size 1.27 1.27)))
+    )
+    (property "Footprint" "" (at 82.55 57.15 0)
+      (effects (font (size 1.27 1.27)) hide)
+    )
+    (property "Datasheet" "" (at 82.55 57.15 0)
+      (effects (font (size 1.27 1.27)) hide)
+    )
