File: projects/03-PIC16F_LCD16x2/KiCad/pic16F887_lcd16x2.kicad_sch (KiCad schematic)
At the start: 5 parts, among them U1 PIC16F887-IP, U2 LCD-016N002L

Commit message: Doc
Parts:
- removed C1: 10uF, symbol Device:C_Polarized
- R1: value 12K -> 10K
Other:
- moved on the sheet: R1, RV1, U1, U2
