File: projects/05-PWM-SPEED-COOLER/KiCad/pic16F628A.kicad_sch (KiCad schematic)
At the start: 6 parts, among them M1 DC Motor, Q1 2N2222, U1 PIC16F628A-IP

Commit message: Doc
Parts:
- removed C1: 10uF, symbol Device:C_Polarized
- R1: value 12K -> 10K
Changed lines of the file:
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@@
     (company "Ricardo Lima Caratti")
   )
-  (junction (at 54.61 29.21) (diameter 0) (color 0 0 0 0)
-  )
   (junction (at 113.03 31.75) (diameter 0) (color 0 0 0 0)
-  )
-  (junction (at 96.52 29.21) (diameter 0) (color 0 0 0 0)
   )
   (wire (pts (xy 22.86 57.15) (xy 22.86 69.85))
@@
     (stroke (width 0) (type default))
   )
-  (wire (pts (xy 101.6 31.75) (xy 96.52 31.75))
-    (stroke (width 0) (type default))
-  )
   (wire (pts (xy 54.61 62.23) (xy 54.61 82.55))
     (stroke (width 0) (type default))
   )
-  (wire (pts (xy 109.22 31.75) (xy 113.03 31.75))
-    (stroke (width 0) (type default))
-  )
   (wire (pts (xy 160.02 31.75) (xy 113.03 31.75))
-    (stroke (width 0) (type default))
-  )
-  (wire (pts (xy 54.61 29.21) (xy 96.52 29.21))
     (stroke (width 0) (type default))
   )
@@
     (stroke (width 0) (type default))
   )
-  (wire (pts (xy 96.52 29.21) (xy 96.52 31.75))
-    (stroke (width 0) (type default))
-  )
   (wire (pts (xy 54.61 29.21) (xy 54.61 52.07))
     (stroke (width 0) (type default))
@@
       (effects (font (size 1.27 1.27)))
     )
-    (property "Value" "12K" (at 156.21 58.42 90)
+    (property "Value" "10K" (at 156.21 58.42 90)
       (effects (font (size 1.27 1.27)))
     )
@@
         (path "/73c37809-7617-4b9f-a70a-5c31575fa255"
           (reference "Q1") (unit 1)
-        )
-      )
-    )
-  )
-  (symbol (lib_id "Device:C_Polarized") (at 105.41 31.75 270) (unit 1)
-    (in_bom yes) (on_board yes) (dnp no) (fields_autoplaced)
-    (property "Reference" "C1" (at 106.299 24.13 90)
-      (effects (font (size 1.27 1.27)))
-    )
-    (property "Value" "10uF" (at 106.299 26.67 90)
-      (effects (font (size 1.27 1.27)))
-    )
-    (property "Footprint" "" (at 101.6 32.7152 0)
-      (effects (font (size 1.27 1.27)) hide)
-    )
-    (property "Datasheet" "~" (at 105.41 31.75 0)
-      (effects (font (size 1.27 1.27)) hide)
-    )
-    (pin "1")
-    (pin "2")
-    (instances
-      (project "pic16F628A"
-        (path "/73c37809-7617-4b9f-a70a-5c31575fa255"
-          (reference "C1") (unit 1)
         )
       )
@@
         )
       )
-    )
-  )
-  (symbol (lib_id "power:GND") (at 96.52 29.21 180) (unit 1)
-    (in_bom yes) (on_board yes) (dnp no) (fields_autoplaced)
-    (property "Reference" "#PWR04" (at 96.52 22.86 0)
-      (effects (font (size 1.27 1.27)) hide)
-    )
-    (property "Value" "GND" (at 96.52 24.13 0)
-      (effects (font (size 1.27 1.27)))
-    )
-    (property "Footprint" "" (at 96.52 29.21 0)
-      (effects (font (size 1.27 1.27)) hide)
-    )
-    (property "Datasheet" "" (at 96.52 29.21 0)
-      (effects (font (size 1.27 1.27)) hide)
-    )
-    (pin "1")
-    (instances
-      (project "pic16F628A"
-        (path "/73c37809-7617-4b9f-a70a-5c31575fa255"
-          (reference "#PWR04") (unit 1)
-        )
-      )
