File: projects/05-PWM-SPEED-COOLER/KiCad/pic16F887_analog_read.kicad_sch (KiCad schematic)
At the start: 6 parts, among them M1 DC Motor, Q1 2N2222, U1 PIC16F887-IP

Commit message: Doc
Parts:
- R1: value 12K -> 10K
Connections:
- net VCC: now also U1.11 (VDD), U1.32 (VDD)
Changed lines of the file:
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@@
     (company "Ricardo Lima Caratti")
   )
+  (junction (at 123.19 31.75) (diameter 0) (color 0 0 0 0)
+  )
   (junction (at 74.93 111.76) (diameter 0) (color 0 0 0 0)
+  )
+  (junction (at 72.39 35.56) (diameter 0) (color 0 0 0 0)
   )
   (wire (pts (xy 38.1 27.94) (xy 38.1 36.83))
@@
     (stroke (width 0) (type default))
   )
+  (wire (pts (xy 72.39 35.56) (xy 74.93 35.56))
+    (stroke (width 0) (type default))
+  )
   (wire (pts (xy 133.35 66.04) (xy 147.32 66.04))
     (stroke (width 0) (type default))
@@
     (stroke (width 0) (type default))
   )
+  (wire (pts (xy 72.39 31.75) (xy 123.19 31.75))
+    (stroke (width 0) (type default))
+  )
   (wire (pts (xy 74.93 111.76) (xy 74.93 119.38))
     (stroke (width 0) (type default))
   )
+  (wire (pts (xy 123.19 31.75) (xy 123.19 39.37))
+    (stroke (width 0) (type default))
+  )
   (wire (pts (xy 125.73 88.9) (xy 123.19 88.9))
+    (stroke (width 0) (type default))
+  )
+  (wire (pts (xy 72.39 35.56) (xy 72.39 31.75))
     (stroke (width 0) (type default))
   )
@@
     (stroke (width 0) (type default))
   )
-  (wire (pts (xy 123.19 29.21) (xy 123.19 39.37))
+  (wire (pts (xy 123.19 29.21) (xy 123.19 31.75))
     (stroke (width 0) (type default))
   )
@@
       (effects (font (size 1.27 1.27)))
     )
-    (property "Value" "12K" (at 41.91 33.02 90)
+    (property "Value" "10K" (at 41.91 33.02 90)
       (effects (font (size 1.27 1.27)))
     )
