File: projects/05-PWM-SPEED-COOLER/KiCad/pic16F887_analog_read_4_wire_cooler .kicad_sch (KiCad schematic)
At the start: 5 parts, among them U1 PIC16F887-IP

Commit message: Documentation
Parts:
- removed RV1: 10K, symbol Device:R_Potentiometer
- added U2: LM35-LP, Package_TO_SOT_THT:TO-92_Inline, symbol Sensor_Temperature:LM35-LP
- Cooler: value (none) -> ~
Connections:
- net GND: now also U2.3 (GND)
- net VCC: now also U2.1 (+V_{S})
- net at U1.2 (C12IN0-/ULPWU/AN0/RA0): now also U2.2 (V_{OUT})
Changed lines of the file:
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@@
+    (stroke (width 0) (type default))
+  )
+  (wire (pts (xy 128.27 50.8) (xy 128.27 58.42))
     (stroke (width 0) (type default))
   )
@@
     (stroke (width 0) (type default))
   )
+  (wire (pts (xy 102.87 43.18) (xy 118.11 43.18))
+    (stroke (width 0) (type default))
+  )
   (wire (pts (xy 123.19 88.9) (xy 135.89 88.9))
     (stroke (width 0) (type default))
   )
-  (wire (pts (xy 102.87 43.18) (xy 119.38 43.18))
+  (wire (pts (xy 128.27 27.94) (xy 128.27 35.56))
     (stroke (width 0) (type default))
   )
@@
     (stroke (width 0) (type default))
   )
-  (wire (pts (xy 123.19 29.21) (xy 123.19 39.37))
-    (stroke (width 0) (type default))
-  )
   (wire (pts (xy 45.72 43.18) (xy 46.99 43.18))
-    (stroke (width 0) (type default))
-  )
-  (wire (pts (xy 123.19 46.99) (xy 123.19 50.8))
     (stroke (width 0) (type default))
   )
@@
     (effects (font (size 1.27 1.27)) (justify left bottom))
   )
+  (symbol (lib_id "Sensor_Temperature:LM35-LP") (at 128.27 43.18 0) (mirror y) (unit 1)
+    (in_bom yes) (on_board yes) (dnp no)
+    (property "Reference" "U2" (at 137.16 41.91 0)
+      (effects (font (size 1.27 1.27)) (justify right))
+    )
+    (property "Value" "LM35-LP" (at 137.16 44.45 0)
+      (effects (font (size 1.27 1.27)) (justify right))
+    )
+    (property "Footprint" "Package_TO_SOT_THT:TO-92_Inline" (at 127 49.53 0)
+      (effects (font (size 1.27 1.27)) (justify left) hide)
+    )
+    (property "Datasheet" "http://www.ti.com/lit/ds/symlink/lm35.pdf" (at 128.27 43.18 0)
+      (effects (font (size 1.27 1.27)) hide)
+    )
+    (pin "1")
+    (pin "2")
+    (pin "3")
+    (instances
+      (project "pic16F887_analog_read_4_wire_cooler "
+        (path "/73c37809-7617-4b9f-a70a-5c31575fa255"
+          (reference "U2") (unit 1)
+        )
+      )
+    )
+  )
   (symbol (lib_id "power:VCC") (at 143.51 76.2 0) (unit 1)
     (in_bom yes) (on_board yes) (dnp no) (fields_autoplaced)
@@
     )
   )
-  (symbol (lib_id "power:VCC") (at 123.19 29.21 0) (unit 1)
-    (in_bom yes) (on_board yes) (dnp no) (fields_autoplaced)
-    (property "Reference" "#12V03" (at 123.19 33.02 0)
-      (effects (font (size 1.27 1.27)) hide)
-    )
-    (property "Value" "VCC" (at 123.19 24.13 0)
-      (effects (font (size 1.27 1.27)))
-    )
-    (property "Footprint" "" (at 123.19 29.21 0)
-      (effects (font (size 1.27 1.27)) hide)
-    )
-    (property "Datasheet" "" (at 123.19 29.21 0)
-      (effects (font (size 1.27 1.27)) hide)
-    )
-    (pin "1")
-    (instances
-      (project "pic16F887_analog_read_4_wire_cooler "
-        (path "/73c37809-7617-4b9f-a70a-5c31575fa255"
-          (reference "#12V03") (unit 1)
-        )
-      )
-    )
-  )
   (symbol (lib_id "Device:R_US") (at 41.91 36.83 90) (unit 1)
     (in_bom yes) (on_board yes) (dnp no) (fields_autoplaced)
@@
     )
   )
-  (symbol (lib_id "power:GND") (at 123.19 50.8 0) (unit 1)
-    (in_bom yes) (on_board yes) (dnp no) (fields_autoplaced)
-    (property "Reference" "#PWR01" (at 123.19 57.15 0)
-      (effects (font (size 1.27 1.27)) hide)
-    )
-    (property "Value" "GND" (at 123.19 55.88 0)
-      (effects (font (size 1.27 1.27)))
-    )
-    (property "Footprint" "" (at 123.19 50.8 0)
-      (effects (font (size 1.27 1.27)) hide)
-    )
-    (property "Datasheet" "" (at 123.19 50.8 0)
+  (symbol (lib_id "power:GND") (at 128.27 58.42 0) (unit 1)
+    (in_bom yes) (on_board yes) (dnp no) (fields_autoplaced)
+    (property "Reference" "#PWR01" (at 128.27 64.77 0)
+      (effects (font (size 1.27 1.27)) hide)
+    )
+    (property "Value" "GND" (at 128.27 63.5 0)
+      (effects (font (size 1.27 1.27)))
+    )
+    (property "Footprint" "" (at 128.27 58.42 0)
+      (effects (font (size 1.27 1.27)) hide)
+    )
+    (property "Datasheet" "" (at 128.27 58.42 0)
       (effects (font (size 1.27 1.27)) hide)
     )
@@
     )
   )
+  (symbol (lib_id "power:VCC") (at 128.27 27.94 0) (unit 1)
+    (in_bom yes) (on_board yes) (dnp no) (fields_autoplaced)
+    (property "Reference" "#12V03" (at 128.27 31.75 0)
+      (effects (font (size 1.27 1.27)) hide)
+    )
+    (property "Value" "VCC" (at 128.27 22.86 0)
+      (effects (font (size 1.27 1.27)))
+    )
+    (property "Footprint" "" (at 128.27 27.94 0)
+      (effects (font (size 1.27 1.27)) hide)
+    )
+    (property "Datasheet" "" (at 128.27 27.94 0)
+      (effects (font (size 1.27 1.27)) hide)
+    )
+    (pin "1")
+    (instances
+      (project "pic16F887_analog_read_4_wire_cooler "
+        (path "/73c37809-7617-4b9f-a70a-5c31575fa255"
+          (reference "#12V03") (unit 1)
+        )
+      )
+    )
+  )
   (symbol (lib_id "Device:R") (at 119.38 88.9 90) (unit 1)
     (in_bom yes) (on_board yes) (dnp no)
@@
       (effects (font (size 1.27 1.27)) (justify left))
     )
-    (property "Value" "" (at 148.59 87.63 0)
+    (property "Value" "~" (at 148.59 87.63 0)
       (effects (font (size 1.27 1.27)) (justify left))
     )
@@
         )
       )
-    )
-  )
-  (symbol (lib_id "Device:R_Potentiometer") (at 123.19 43.18 180) (unit 1)
-    (in_bom yes) (on_board yes) (dnp no) (fields_autoplaced)
-    (property "Reference" "RV1" (at 125.73 41.91 0)
-      (effects (font (size 1.27 1.27)) (justify right))
-    )
-    (property "Value" "10K" (at 125.73 44.45 0)
-      (effects (font (size 1.27 1.27)) (justify right))
-    )
-    (property "Footprint" "" (at 123.19 43.18 0)
-      (effects (font (size 1.27 1.27)) hide)
-    )
-    (property "Datasheet" "~" (at 123.19 43.18 0)
-      (effects (font (size 1.27 1.27)) hide)
-    )
-    (pin "1")
-    (pin "2")
-    (pin "3")
-    (instances
-      (project "pic16F887_analog_read_4_wire_cooler "
-        (path "/73c37809-7617-4b9f-a70a-5c31575fa255"
-          (reference "RV1") (unit 1)
-        )
-      )

Commit message: Documentation
Parts:
- added R3: 12K, symbol Device:R_US
Connections:
- net VCC: now also R3.2
- net at U1.33 (INT/AN12/RB0): now also Cooler.3 (Tacho), R3.1
Changed lines of the file:
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@@
   (junction (at 74.93 111.76) (diameter 0) (color 0 0 0 0)
   )
+  (junction (at 127 83.82) (diameter 0) (color 0 0 0 0)
+  )
   (wire (pts (xy 38.1 27.94) (xy 38.1 36.83))
     (stroke (width 0) (type default))
   )
+  (wire (pts (xy 127 83.82) (xy 135.89 83.82))
+    (stroke (width 0) (type default))
+  )
   (wire (pts (xy 102.87 88.9) (xy 115.57 88.9))
     (stroke (width 0) (type default))
   )
+  (wire (pts (xy 119.38 83.82) (xy 127 83.82))
+    (stroke (width 0) (type default))
+  )
   (wire (pts (xy 143.51 76.2) (xy 143.51 78.74))
     (stroke (width 0) (type default))
@@
     (stroke (width 0) (type default))
   )
+  (wire (pts (xy 119.38 60.96) (xy 119.38 83.82))
+    (stroke (width 0) (type default))
+  )
   (wire (pts (xy 102.87 43.18) (xy 118.11 43.18))
     (stroke (width 0) (type default))
@@
     (stroke (width 0) (type default))
   )
+  (wire (pts (xy 102.87 60.96) (xy 119.38 60.96))
+    (stroke (width 0) (type default))
+  )
   (wire (pts (xy 72.39 111.76) (xy 74.93 111.76))
     (stroke (width 0) (type default))
   )
+  (wire (pts (xy 127 71.12) (xy 127 73.66))
+    (stroke (width 0) (type default))
+  )
   (wire (pts (xy 143.51 91.44) (xy 143.51 111.76))
     (stroke (width 0) (type default))
   )
   (wire (pts (xy 45.72 36.83) (xy 45.72 43.18))
+    (stroke (width 0) (type default))
+  )
+  (wire (pts (xy 127 81.28) (xy 127 83.82))
     (stroke (width 0) (type default))
   )
@@
     )
   )
+  (symbol (lib_id "Device:R_US") (at 127 77.47 180) (unit 1)
+    (in_bom yes) (on_board yes) (dnp no) (fields_autoplaced)
+    (property "Reference" "R3" (at 129.54 76.2 0)
+      (effects (font (size 1.27 1.27)) (justify right))
+    )
+    (property "Value" "12K" (at 129.54 78.74 0)
+      (effects (font (size 1.27 1.27)) (justify right))
+    )
+    (property "Footprint" "" (at 125.984 77.216 90)
+      (effects (font (size 1.27 1.27)) hide)
+    )
+    (property "Datasheet" "~" (at 127 77.47 0)
+      (effects (font (size 1.27 1.27)) hide)
+    )
+    (pin "1")
+    (pin "2")
+    (instances
+      (project "pic16F887_analog_read_4_wire_cooler "
+        (path "/73c37809-7617-4b9f-a70a-5c31575fa255"
+          (reference "R3") (unit 1)
+        )
+      )
+    )
+  )
   (symbol (lib_id "power:VCC") (at 38.1 27.94 0) (unit 1)
     (in_bom yes) (on_board yes) (dnp no) (fields_autoplaced)
@@
         )
       )
+    )
+  )
+  (symbol (lib_id "power:VCC") (at 127 71.12 0) (unit 1)
+    (in_bom yes) (on_board yes) (dnp no) (fields_autoplaced)
+    (property "Reference" "#12V04" (at 127 74.93 0)
+      (effects (font (size 1.27 1.27)) hide)
+    )
+    (property "Value" "VCC" (at 127 66.04 0)
+      (effects (font (size 1.27 1.27)))
+    )
+    (property "Footprint" "" (at 127 71.12 0)
+      (effects (font (size 1.27 1.27)) hide)
+    )
+    (property "Datasheet" "" (at 127 71.12 0)
+      (effects (font (size 1.27 1.27)) hide)
+    )
+    (pin "1")
+    (instances
+      (project "pic16F887_analog_read_4_wire_cooler "
+        (path "/73c37809-7617-4b9f-a70a-5c31575fa255"
+          (reference "#12V04") (unit 1)
+        )
+      )

Commit message: Doc
Parts:
- R1: value 12K -> 10K
Connections:
- net VCC: now also U1.11 (VDD), U1.32 (VDD)
Changed lines of the file:
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@@
   (junction (at 127 83.82) (diameter 0) (color 0 0 0 0)
   )
+  (junction (at 73.66 35.56) (diameter 0) (color 0 0 0 0)
+  )
+  (junction (at 128.27 30.48) (diameter 0) (color 0 0 0 0)
+  )
   (wire (pts (xy 38.1 27.94) (xy 38.1 36.83))
+    (stroke (width 0) (type default))
+  )
+  (wire (pts (xy 128.27 30.48) (xy 128.27 35.56))
+    (stroke (width 0) (type default))
+  )
+  (wire (pts (xy 72.39 35.56) (xy 73.66 35.56))
     (stroke (width 0) (type default))
   )
@@
   )
   (wire (pts (xy 102.87 88.9) (xy 115.57 88.9))
+    (stroke (width 0) (type default))
+  )
+  (wire (pts (xy 73.66 30.48) (xy 128.27 30.48))
     (stroke (width 0) (type default))
   )
@@
     (stroke (width 0) (type default))
   )
+  (wire (pts (xy 73.66 35.56) (xy 74.93 35.56))
+    (stroke (width 0) (type default))
+  )
   (wire (pts (xy 119.38 60.96) (xy 119.38 83.82))
     (stroke (width 0) (type default))
@@
     (stroke (width 0) (type default))
   )
-  (wire (pts (xy 128.27 27.94) (xy 128.27 35.56))
+  (wire (pts (xy 128.27 27.94) (xy 128.27 30.48))
     (stroke (width 0) (type default))
   )
@@
   )
   (wire (pts (xy 143.51 91.44) (xy 143.51 111.76))
+    (stroke (width 0) (type default))
+  )
+  (wire (pts (xy 73.66 35.56) (xy 73.66 30.48))
     (stroke (width 0) (type default))
   )
@@
       (effects (font (size 1.27 1.27)))
     )
-    (property "Value" "12K" (at 41.91 33.02 90)
+    (property "Value" "10K" (at 41.91 33.02 90)
       (effects (font (size 1.27 1.27)))
     )
