File: projects/07-HC-S04-URTASONIC/KiCad/PIC10F200_HC_S04_1led.kicad_sch (KiCad schematic)
At the start: 4 parts, among them U1 PIC12F675-IP, U2 HC-SR04

Commit message: Doc
Parts:
- removed U1: PIC12F675-IP, Package_DIP:DIP-8_W7.62mm, symbol MCU_Microchip_PIC12:PIC12F675-IP
- added R1: 10K, symbol Device:R
- added U1: PIC10F200-IP, Package_DIP:DIP-8_W7.62mm, symbol MCU_Microchip_PIC10:PIC10F200-IP
Connections:
- net +5V: now also R1.2, U1.2 (VDD)
- net GND: now also D1.1 (K), U1.7 (VSS)
- net at U2.2 (TRIG): now also U1.4 (GP1)
- net at U2.3 (ECHO): now also U1.3 (GP2)
- net at R2.2: now also U1.5 (GP0)
- new net: R1.1, U1.8 (GP3)
Other:
- note removed: "Green"
- moved on the sheet: D1, R2
