File: projects/07-HC-S04-URTASONIC/KiCad/PIC12F675_HC_S04_3led.kicad_sch (KiCad schematic)
At the start: 8 parts, among them U1 PIC12F675-IP, U2 HC-SR04

Commit message: Doc
Parts:
- added R1: 10K, symbol Device:R
Connections:
- net +5V: now also R1.2
- net at U1.4 (GP3): now also R1.1
Other:
- title: PIC16F628A for Beginners - 1 -> PIC12F675 and HC-S04
- moved on the sheet: D1, D2, D3, R2, R3, R4, U1, U2
