File: projects/07-HC-S04-URTASONIC/KiCad/PIC16F628A_LED_RGB_COMMON_ULTRASONIC.kicad_sch (KiCad schematic)
At the start: 6 parts, among them U1 PIC16F628A-IP, U2 HC-SR04

Commit message: Documentation
Parts:
- added R4: 12K, symbol Device:R
Connections:
- net VCC: now also R4.2
- net at U1.4 (~{MCLR}/Vpp/RA5): now also R4.1
Changed lines of the file:
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@@
   (junction (at 100.33 31.75) (diameter 0) (color 0 0 0 0)
   )
+  (wire (pts (xy 139.7 54.61) (xy 142.24 54.61))
+    (stroke (width 0) (type default))
+  )
   (wire (pts (xy 100.33 31.75) (xy 100.33 34.29))
     (stroke (width 0) (type default))
@@
     (stroke (width 0) (type default))
   )
+  (wire (pts (xy 142.24 52.07) (xy 142.24 54.61))
+    (stroke (width 0) (type default))
+  )
   (wire (pts (xy 149.86 72.39) (xy 100.33 72.39))
     (stroke (width 0) (type default))
   )
   (wire (pts (xy 128.27 44.45) (xy 149.86 44.45))
+    (stroke (width 0) (type default))
+  )
+  (wire (pts (xy 128.27 54.61) (xy 132.08 54.61))
     (stroke (width 0) (type default))
   )
@@
     (pin "2")
     (instances
-      (project "LED_RGB_COMMON_ULTRASONIC"
+      (project "PIC16F628A_LED_RGB_COMMON_ULTRASONIC"
         (path "/261f22d7-9959-48cd-bc20-0bbce393e6d1"
           (reference "R3") (unit 1)
@@
     (pin "2")
     (instances
-      (project "LED_RGB_COMMON_ULTRASONIC"
+      (project "PIC16F628A_LED_RGB_COMMON_ULTRASONIC"
         (path "/261f22d7-9959-48cd-bc20-0bbce393e6d1"
           (reference "R2") (unit 1)
@@
     (pin "4")
     (instances
-      (project "LED_RGB_COMMON_ULTRASONIC"
+      (project "PIC16F628A_LED_RGB_COMMON_ULTRASONIC"
         (path "/261f22d7-9959-48cd-bc20-0bbce393e6d1"
           (reference "U2") (unit 1)
@@
     (pin "9")
     (instances
-      (project "LED_RGB_COMMON_ULTRASONIC"
+      (project "PIC16F628A_LED_RGB_COMMON_ULTRASONIC"
         (path "/261f22d7-9959-48cd-bc20-0bbce393e6d1"
           (reference "U1") (unit 1)
+        )
+      )
+    )
+  )
+  (symbol (lib_id "Device:R") (at 135.89 54.61 90) (unit 1)
+    (in_bom yes) (on_board yes) (dnp no) (fields_autoplaced)
+    (property "Reference" "R4" (at 135.89 48.26 90)
+      (effects (font (size 1.27 1.27)))
+    )
+    (property "Value" "12K" (at 135.89 50.8 90)
+      (effects (font (size 1.27 1.27)))
+    )
+    (property "Footprint" "" (at 135.89 56.388 90)
+      (effects (font (size 1.27 1.27)) hide)
+    )
+    (property "Datasheet" "~" (at 135.89 54.61 0)
+      (effects (font (size 1.27 1.27)) hide)
+    )
+    (pin "1")
+    (pin "2")
+    (instances
+      (project "PIC16F628A_LED_RGB_COMMON_ULTRASONIC"
+        (path "/261f22d7-9959-48cd-bc20-0bbce393e6d1"
+          (reference "R4") (unit 1)
         )
       )
@@
     (pin "4")
     (instances
-      (project "LED_RGB_COMMON_ULTRASONIC"
+      (project "PIC16F628A_LED_RGB_COMMON_ULTRASONIC"
         (path "/261f22d7-9959-48cd-bc20-0bbce393e6d1"
           (reference "D1") (unit 1)
@@
     )
   )
+  (symbol (lib_id "power:VCC") (at 142.24 52.07 0) (unit 1)
+    (in_bom yes) (on_board yes) (dnp no) (fields_autoplaced)
+    (property "Reference" "#PWR01" (at 142.24 55.88 0)
+      (effects (font (size 1.27 1.27)) hide)
+    )
+    (property "Value" "VCC" (at 142.24 46.99 0)
+      (effects (font (size 1.27 1.27)))
+    )
+    (property "Footprint" "" (at 142.24 52.07 0)
+      (effects (font (size 1.27 1.27)) hide)
+    )
+    (property "Datasheet" "" (at 142.24 52.07 0)
+      (effects (font (size 1.27 1.27)) hide)
+    )
+    (pin "1")
+    (instances
+      (project "PIC16F628A_LED_RGB_COMMON_ULTRASONIC"
+        (path "/261f22d7-9959-48cd-bc20-0bbce393e6d1"
+          (reference "#PWR01") (unit 1)
+        )
+      )
+    )
+  )
   (symbol (lib_id "power:GND") (at 100.33 74.93 0) (unit 1)
     (in_bom yes) (on_board yes) (dnp no) (fields_autoplaced)
@@
     (pin "1")
     (instances
-      (project "LED_RGB_COMMON_ULTRASONIC"
+      (project "PIC16F628A_LED_RGB_COMMON_ULTRASONIC"
         (path "/261f22d7-9959-48cd-bc20-0bbce393e6d1"
           (reference "#PWR03") (unit 1)
@@
     (pin "1")
     (instances
-      (project "LED_RGB_COMMON_ULTRASONIC"
+      (project "PIC16F628A_LED_RGB_COMMON_ULTRASONIC"
         (path "/261f22d7-9959-48cd-bc20-0bbce393e6d1"
           (reference "#PWR02") (unit 1)
@@
     (pin "2")
     (instances
-      (project "LED_RGB_COMMON_ULTRASONIC"
+      (project "PIC16F628A_LED_RGB_COMMON_ULTRASONIC"
         (path "/261f22d7-9959-48cd-bc20-0bbce393e6d1"
           (reference "R1") (unit 1)

Commit message: Doc
Parts:
- R4: value 12K -> 10K
Changed lines of the file:
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@@
 (kicad_sch (version 20230121) (generator eeschema)
-  (paper "User" 203.2 152.4)
+  (paper "User" 180.01 129.997)
   (title_block
     (title "Distance Alert - PIC16F628A with HC-SR04 and RGB LED")
@@
       (effects (font (size 1.27 1.27)))
     )
-    (property "Value" "12K" (at 135.89 50.8 90)
-      (effects (font (size 1.27 1.27)))
-    )
+    (property "Value" "10K" (at 135.89 50.8 90)
+      (effects (font (size 1.27 1.27)))
+    )
