File: projects/07-HC-S04-URTASONIC/KiCad/PIC16F876A_LCD_ULTRASONIC copy.kicad_sch (KiCad schematic)
At the start: 8 parts, among them U1 PIC16F876-XXISO, U2 HC-SR04, U3 LCD-16x2, Y1 4MHz

Commit message: Doc
Parts:
- R1: value 12K -> 10K
Other:
- moved on the sheet: C1, C2, R1, RV1, U1, U2, U3, Y1
