File: projects/08-LM35_OR_TMP36/KiCad/PIC12F675_lm35_3led.kicad_sch (KiCad schematic)
At the start: 9 parts, among them U1 PIC12F675-IP, U2 LM35-LP

Commit message: Doc
Parts:
- R1: value 12K -> 10K
Other:
- title: PIC16F628A for Beginners - 1 -> PIC12F675 and LM35
- moved on the sheet: D1, D2, D3, R1, R2, R3, R4, U1, U2
