File: projects/08-LM35_OR_TMP36/KiCad/PIC12F675_lm35_led.kicad_sch (KiCad schematic)
At the start: 7 parts, among them U1 PIC12F675-IP, U2 LM35-LP

Commit message: Doc
Parts:
- removed C1: 10uF, symbol Device:C_Polarized
- removed C2: 100nF, symbol Device:C
- R1: value 12K -> 10K
Other:
- title: PIC16F628A for Beginners - 1 -> PIC12F675 and LM35
- moved on the sheet: D1, R1, R2, U1, U2
