File: projects/09-LDR_PHOTOCELL/KiCad/PIC12F675_LDR.kicad_sch (KiCad schematic)
At the start: 7 parts, among them Q1 NPN, U1 PIC12F675-IP

Commit message: Doc
Parts:
- R1: value 12K -> 10K
Other:
- note added: "Driver"
- moved on the sheet: D1, Q1, R1, R2, R3, R4, U1
