File: projects/12-ONE_WIRE_PROTOCOL/PIC10F200/KiCad/PIC10F200_1_wire_DS18B20.kicad_sch (KiCad schematic)
At the start: 8 parts, among them U1 PIC10F200-IP, U2 DS18B20

Commit message: Doc
Parts:
- removed D2: LED, symbol Device:LED
- removed R2: 360R, symbol Device:R
Connections:
- net GND: now also R3.1; no longer D1.1 (K)
- net at U1.4 (GP1): now also D1.1 (K); no longer R3.1
Other:
- note removed: "GP1 HIGH and GP2 LOW = HOT GP1 LOW and GP2 HIG = COLD GP1 and GP2 LOW = REGULAR"
- moved on the sheet: D1, R1, R10, R3, U1, U2
