File: projects/12-ONE_WIRE_PROTOCOL/PIC16F887/KiCad/pic16F887_ds18b20_lcd16x2.kicad_sch (KiCad schematic)
At the start: 5 parts, among them U1 PIC16F887-IP, U2 LCD-016N002L, U3 DS18B20

Commit message: Doc
Parts:
- added R2: 4.7K, symbol Device:R_US
Connections:
- net +5V: now also R2.2
- net at U1.33 (INT/AN12/RB0), U3.2 (DQ): now also R2.1
Changed lines of the file:
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@@
     (company "Ricardo Lima Caratti")
   )
+  (junction (at 120.65 33.02) (diameter 0) (color 0 0 0 0)
+  )
   (junction (at 132.08 33.02) (diameter 0) (color 0 0 0 0)
   )
@@
   (junction (at 143.51 110.49) (diameter 0) (color 0 0 0 0)
   )
+  (junction (at 123.19 41.91) (diameter 0) (color 0 0 0 0)
+  )
   (junction (at 132.08 59.69) (diameter 0) (color 0 0 0 0)
   )
@@
     (stroke (width 0) (type default))
   )
+  (wire (pts (xy 120.65 33.02) (xy 83.82 33.02))
+    (stroke (width 0) (type default))
+  )
   (wire (pts (xy 143.51 64.77) (xy 143.51 33.02))
     (stroke (width 0) (type default))
@@
     (stroke (width 0) (type default))
   )
+  (wire (pts (xy 120.65 41.91) (xy 123.19 41.91))
+    (stroke (width 0) (type default))
+  )
   (wire (pts (xy 177.8 66.04) (xy 177.8 33.02))
     (stroke (width 0) (type default))
@@
     (stroke (width 0) (type default))
   )
+  (wire (pts (xy 120.65 33.02) (xy 120.65 34.29))
+    (stroke (width 0) (type default))
+  )
   (wire (pts (xy 111.76 97.79) (xy 133.35 97.79))
     (stroke (width 0) (type default))
@@
     (stroke (width 0) (type default))
   )
+  (wire (pts (xy 111.76 59.69) (xy 123.19 59.69))
+    (stroke (width 0) (type default))
+  )
   (wire (pts (xy 153.67 77.47) (xy 163.83 77.47))
     (stroke (width 0) (type default))
@@
     (stroke (width 0) (type default))
   )
-  (wire (pts (xy 111.76 59.69) (xy 123.19 59.69))
-    (stroke (width 0) (type default))
-  )
   (wire (pts (xy 143.51 33.02) (xy 132.08 33.02))
     (stroke (width 0) (type default))
@@
     (stroke (width 0) (type default))
   )
-  (wire (pts (xy 132.08 33.02) (xy 83.82 33.02))
+  (wire (pts (xy 132.08 33.02) (xy 120.65 33.02))
     (stroke (width 0) (type default))
   )
@@
     (pin "K2")
     (instances
-      (project "pic16F887_lcd16x2"
+      (project "pic16F887_ds18b20_lcd16x2"
         (path "/73c37809-7617-4b9f-a70a-5c31575fa255"
           (reference "U2") (unit 1)
@@
     (pin "2")
     (instances
-      (project "pic16F887_lcd16x2"
+      (project "pic16F887_ds18b20_lcd16x2"
         (path "/73c37809-7617-4b9f-a70a-5c31575fa255"
           (reference "R1") (unit 1)
@@
     (pin "1")
     (instances
-      (project "pic16F887_lcd16x2"
+      (project "pic16F887_ds18b20_lcd16x2"
         (path "/73c37809-7617-4b9f-a70a-5c31575fa255"
           (reference "#PWR03") (unit 1)
@@
     (pin "9")
     (instances
-      (project "pic16F887_lcd16x2"
+      (project "pic16F887_ds18b20_lcd16x2"
         (path "/73c37809-7617-4b9f-a70a-5c31575fa255"
           (reference "U1") (unit 1)
@@
     )
   )
+  (symbol (lib_id "Device:R_US") (at 120.65 38.1 180) (unit 1)
+    (in_bom yes) (on_board yes) (dnp no)
+    (property "Reference" "R2" (at 114.3 38.1 90)
+      (effects (font (size 1.27 1.27)))
+    )
+    (property "Value" "4.7K" (at 116.84 38.1 90)
+      (effects (font (size 1.27 1.27)))
+    )
+    (property "Footprint" "" (at 119.634 37.846 90)
+      (effects (font (size 1.27 1.27)) hide)
+    )
+    (property "Datasheet" "~" (at 120.65 38.1 0)
+      (effects (font (size 1.27 1.27)) hide)
+    )
+    (pin "1")
+    (pin "2")
+    (instances
+      (project "pic16F887_ds18b20_lcd16x2"
+        (path "/73c37809-7617-4b9f-a70a-5c31575fa255"
+          (reference "R2") (unit 1)
+        )
+      )
+    )
+  )
   (symbol (lib_id "power:+5V") (at 83.82 25.4 0) (unit 1)
     (in_bom yes) (on_board yes) (dnp no)
@@
     (pin "1")
     (instances
-      (project "pic16F887_lcd16x2"
+      (project "pic16F887_ds18b20_lcd16x2"
         (path "/73c37809-7617-4b9f-a70a-5c31575fa255"
           (reference "#PWR01") (unit 1)
@@
   (symbol (lib_id "Sensor_Temperature:DS18B20") (at 132.08 41.91 0) (mirror y) (unit 1)
     (in_bom yes) (on_board yes) (dnp no)
-    (property "Reference" "U3" (at 120.65 38.1 0)
+    (property "Reference" "U3" (at 127 34.29 0)
       (effects (font (size 1.27 1.27)) (justify right))
     )
-    (property "Value" "DS18B20" (at 119.38 35.56 0)
+    (property "Value" "DS18B20" (at 133.35 34.29 0)
       (effects (font (size 1.27 1.27)) (justify right))
     )
@@
     (pin "3")
     (instances
-      (project "pic16F887_lcd16x2"
+      (project "pic16F887_ds18b20_lcd16x2"
         (path "/73c37809-7617-4b9f-a70a-5c31575fa255"
           (reference "U3") (unit 1)
@@
     (pin "1")
     (instances
-      (project "pic16F887_lcd16x2"
+      (project "pic16F887_ds18b20_lcd16x2"
         (path "/73c37809-7617-4b9f-a70a-5c31575fa255"
           (reference "#PWR02") (unit 1)
@@
     (pin "3")
     (instances
-      (project "pic16F887_lcd16x2"
+      (project "pic16F887_ds18b20_lcd16x2"
         (path "/73c37809-7617-4b9f-a70a-5c31575fa255"
           (reference "RV1") (unit 1)
