File: projects/14-GAS_SENSOR/PIC16F887/KiCad/pic16F887_MQ_GAS_SENSOR_lcd16x2.kicad_sch (KiCad schematic)
At the start: 5 parts, among them U1 PIC16F887-IP, U2 LCD-016N002L, U3 MQ-2

Commit message: Doc
Parts:
- added R2: 10K, symbol Device:R_US
Connections:
- net +5V: now also U3.2 (VH+), U3.4 (A2), U3.6 (A1)
- net GND: now also U3.5 (VH-), R2.2
- net at U3.1 (B1): now also U3.3 (B2), R2.1
Other:
- note added: "A0"
- note added: "D0"
- note added: "GND"
- note added: "VCC"
Changed lines of the file:
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@@
     (company "Ricardo Lima Caratti")
   )
-  (junction (at 120.65 33.02) (diameter 0) (color 0 0 0 0)
-  )
-  (junction (at 132.08 33.02) (diameter 0) (color 0 0 0 0)
+  (junction (at 26.67 57.15) (diameter 0) (color 0 0 0 0)
+  )
+  (junction (at 36.83 67.31) (diameter 0) (color 0 0 0 0)
   )
   (junction (at 163.83 110.49) (diameter 0) (color 0 0 0 0)
@@
   (junction (at 143.51 110.49) (diameter 0) (color 0 0 0 0)
   )
+  (junction (at 16.51 64.77) (diameter 0) (color 0 0 0 0)
+  )
+  (junction (at 41.91 110.49) (diameter 0) (color 0 0 0 0)
+  )
+  (junction (at 81.28 110.49) (diameter 0) (color 0 0 0 0)
+  )
+  (junction (at 36.83 33.02) (diameter 0) (color 0 0 0 0)
+  )
   (wire (pts (xy 153.67 80.01) (xy 163.83 80.01))
     (stroke (width 0) (type default))
@@
     (stroke (width 0) (type default))
   )
+  (wire (pts (xy 36.83 67.31) (xy 41.91 67.31))
+    (stroke (width 0) (type default))
+  )
+  (wire (pts (xy 36.83 67.31) (xy 36.83 69.85))
+    (stroke (width 0) (type default))
+  )
   (wire (pts (xy 133.35 72.39) (xy 132.08 72.39))
     (stroke (width 0) (type default))
@@
     (stroke (width 0) (type default))
   )
+  (wire (pts (xy 41.91 76.2) (xy 41.91 67.31))
+    (stroke (width 0) (type default))
+  )
   (wire (pts (xy 111.76 90.17) (xy 129.54 90.17))
     (stroke (width 0) (type default))
@@
     (stroke (width 0) (type default))
   )
+  (wire (pts (xy 26.67 77.47) (xy 26.67 110.49))
+    (stroke (width 0) (type default))
+  )
   (wire (pts (xy 143.51 105.41) (xy 143.51 110.49))
     (stroke (width 0) (type default))
   )
-  (wire (pts (xy 120.65 33.02) (xy 83.82 33.02))
-    (stroke (width 0) (type default))
-  )
   (wire (pts (xy 143.51 64.77) (xy 143.51 33.02))
     (stroke (width 0) (type default))
   )
+  (wire (pts (xy 41.91 110.49) (xy 81.28 110.49))
+    (stroke (width 0) (type default))
+  )
   (wire (pts (xy 111.76 92.71) (xy 133.35 92.71))
     (stroke (width 0) (type default))
@@
     (stroke (width 0) (type default))
   )
-  (wire (pts (xy 120.65 33.02) (xy 120.65 34.29))
+  (wire (pts (xy 34.29 59.69) (xy 39.37 59.69))
     (stroke (width 0) (type default))
   )
@@
     (stroke (width 0) (type default))
   )
+  (wire (pts (xy 26.67 57.15) (xy 26.67 33.02))
+    (stroke (width 0) (type default))
+  )
   (wire (pts (xy 132.08 59.69) (xy 134.62 59.69))
     (stroke (width 0) (type default))
   )
+  (wire (pts (xy 81.28 110.49) (xy 83.82 110.49))
+    (stroke (width 0) (type default))
+  )
+  (wire (pts (xy 111.76 82.55) (xy 115.57 82.55))
+    (stroke (width 0) (type default))
+  )
   (wire (pts (xy 44.45 41.91) (xy 55.88 41.91))
     (stroke (width 0) (type default))
@@
     (stroke (width 0) (type default))
   )
-  (wire (pts (xy 81.28 110.49) (xy 83.82 110.49))
+  (wire (pts (xy 26.67 110.49) (xy 41.91 110.49))
+    (stroke (width 0) (type default))
+  )
+  (wire (pts (xy 111.76 41.91) (xy 123.19 41.91))
     (stroke (width 0) (type default))
   )
@@
     (stroke (width 0) (type default))
   )
+  (wire (pts (xy 16.51 57.15) (xy 16.51 64.77))
+    (stroke (width 0) (type default))
+  )
+  (wire (pts (xy 41.91 83.82) (xy 41.91 110.49))
+    (stroke (width 0) (type default))
+  )
+  (wire (pts (xy 16.51 57.15) (xy 26.67 57.15))
+    (stroke (width 0) (type default))
+  )
   (wire (pts (xy 153.67 77.47) (xy 163.83 77.47))
     (stroke (width 0) (type default))
   )
+  (wire (pts (xy 36.83 64.77) (xy 36.83 67.31))
+    (stroke (width 0) (type default))
+  )
   (wire (pts (xy 143.51 33.02) (xy 163.83 33.02))
     (stroke (width 0) (type default))
   )
-  (wire (pts (xy 143.51 33.02) (xy 132.08 33.02))
-    (stroke (width 0) (type default))
-  )
   (wire (pts (xy 129.54 90.17) (xy 129.54 69.85))
     (stroke (width 0) (type default))
   )
-  (wire (pts (xy 132.08 33.02) (xy 132.08 34.29))
+  (wire (pts (xy 16.51 64.77) (xy 16.51 69.85))
     (stroke (width 0) (type default))
   )
@@
     (stroke (width 0) (type default))
   )
+  (wire (pts (xy 26.67 33.02) (xy 36.83 33.02))
+    (stroke (width 0) (type default))
+  )
   (wire (pts (xy 83.82 110.49) (xy 143.51 110.49))
     (stroke (width 0) (type default))
@@
     (stroke (width 0) (type default))
   )
-  (wire (pts (xy 132.08 33.02) (xy 120.65 33.02))
+  (wire (pts (xy 83.82 33.02) (xy 143.51 33.02))
     (stroke (width 0) (type default))
   )
   (wire (pts (xy 36.83 41.91) (xy 36.83 33.02))
     (stroke (width 0) (type default))
+  )
+  (text "A0" (at 121.92 41.91 0)
+    (effects (font (size 1.27 1.27)) (justify left bottom))
+  )
+  (text "D0" (at 115.57 82.55 0)
+    (effects (font (size 1.27 1.27)) (justify left bottom))
+  )
+  (text "D0" (at 39.37 60.96 0)
+    (effects (font (size 1.27 1.27)) (justify left bottom))
+  )
+  (text "A0" (at 39.37 66.04 0)
+    (effects (font (size 1.27 1.27)) (justify left bottom))
+  )
+  (text "VCC" (at 21.59 55.88 0)
+    (effects (font (size 1.27 1.27)) (justify left bottom))
+  )
+  (text "GND" (at 27.94 78.74 0)
+    (effects (font (size 1.27 1.27)) (justify left bottom))
   )
   (symbol (lib_id "Display_Character:LCD-016N002L") (at 143.51 85.09 0) (unit 1)
@@
         )
       )
+    )
+  )
+  (symbol (lib_id "Device:R_US") (at 41.91 80.01 0) (unit 1)
+    (in_bom yes) (on_board yes) (dnp no)
+    (property "Reference" "R2" (at 48.26 80.01 90)
+      (effects (font (size 1.27 1.27)))
+    )
+    (property "Value" "10K" (at 45.72 80.01 90)
+      (effects (font (size 1.27 1.27)))
+    )
+    (property "Footprint" "" (at 42.926 80.264 90)
+      (effects (font (size 1.27 1.27)) hide)
+    )
+    (property "Datasheet" "~" (at 41.91 80.01 0)
+      (effects (font (size 1.27 1.27)) hide)
+    )
+    (pin "1")
+    (pin "2")
+    (instances
+      (project "pic16F887_MQ_GAS_SENSOR_lcd16x2"
+        (path "/73c37809-7617-4b9f-a70a-5c31575fa255"
+          (reference "R2") (unit 1)
+        )
+      )
