File: projects/14-GAS_SENSOR/PIC12F675/KiCad/pic12F675_MQ_GAS_SENSOR_LEDs.kicad_sch (KiCad schematic)
At the start: 10 parts, among them U1 PIC12F675-IP, U3 MQ-2

Commit message: Doc
Connections:
- net at R2.1, U3.1 (B1), U3.3 (B2): no longer U1.7 (GP0)
- net at R3.1: now also U1.7 (GP0); no longer U1.3 (GP4)
Changed lines of the file:
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@@
-    (stroke (width 0) (type default))
-  )
-  (wire (pts (xy 91.44 64.77) (xy 67.31 64.77))
     (stroke (width 0) (type default))
   )
@@
     (stroke (width 0) (type default))
   )
-  (wire (pts (xy 129.54 67.31) (xy 129.54 81.28))
+  (wire (pts (xy 86.36 83.82) (xy 158.75 83.82))
     (stroke (width 0) (type default))
   )
@@
     (stroke (width 0) (type default))
   )
-  (wire (pts (xy 129.54 81.28) (xy 158.75 81.28))
+  (wire (pts (xy 158.75 81.28) (xy 158.75 83.82))
     (stroke (width 0) (type default))
   )
@@
     (stroke (width 0) (type default))
   )
+  (wire (pts (xy 86.36 64.77) (xy 86.36 83.82))
+    (stroke (width 0) (type default))
+  )
+  (wire (pts (xy 91.44 64.77) (xy 86.36 64.77))
+    (stroke (width 0) (type default))
+  )
   (wire (pts (xy 181.61 104.14) (xy 187.96 104.14))
     (stroke (width 0) (type default))
@@
     (effects (font (size 1.27 1.27)) (justify left bottom))
   )
+  (text "A0" (at 130.81 68.58 0)
+    (effects (font (size 1.27 1.27)) (justify left bottom))
+  )
