File: projects/99-Servomotor/KiCad/pic10F200_servo.kicad_sch (KiCad schematic)
At the start: 5 parts, among them M1 Motor_Servo, U1 PIC10F200-IP

Commit message: Doc
Parts:
- added SW1, SW2: SW_Push, symbol Switch:SW_Push
- R2, R3: value 10K -> 1K
Connections:
- net GND: now also SW1.2, SW2.2
- net at R3.1: now also SW2.1
- net at R2.1: now also SW1.1
Other:
- title: Basic Servo Controll with PIC16F628A -> Controlling a Servo with PIC10F200 and push buttons
Changed lines of the file:
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@@
   (paper "User" 200 140.005)
   (title_block
-    (title "Basic Servo Controll with PIC16F628A")
+    (title "Controlling a Servo with PIC10F200 and push buttons")
     (company "Ricardo Lima Caratti")
   )
   (junction (at 66.04 29.21) (diameter 0) (color 0 0 0 0)
   )
+  (junction (at 138.43 57.15) (diameter 0) (color 0 0 0 0)
+  )
   (junction (at 83.82 73.66) (diameter 0) (color 0 0 0 0)
   )
+  (wire (pts (xy 109.22 54.61) (xy 116.84 54.61))
+    (stroke (width 0) (type default))
+  )
   (wire (pts (xy 66.04 29.21) (xy 83.82 29.21))
     (stroke (width 0) (type default))
   )
+  (wire (pts (xy 127 49.53) (xy 138.43 49.53))
+    (stroke (width 0) (type default))
+  )
   (wire (pts (xy 83.82 72.39) (xy 83.82 73.66))
     (stroke (width 0) (type default))
   )
+  (wire (pts (xy 138.43 49.53) (xy 138.43 57.15))
+    (stroke (width 0) (type default))
+  )
   (wire (pts (xy 63.5 73.66) (xy 83.82 73.66))
     (stroke (width 0) (type default))
   )
+  (wire (pts (xy 116.84 49.53) (xy 116.84 54.61))
+    (stroke (width 0) (type default))
+  )
   (wire (pts (xy 83.82 41.91) (xy 83.82 29.21))
     (stroke (width 0) (type default))
@@
     (stroke (width 0) (type default))
   )
+  (wire (pts (xy 116.84 59.69) (xy 116.84 66.04))
+    (stroke (width 0) (type default))
+  )
+  (wire (pts (xy 109.22 59.69) (xy 116.84 59.69))
+    (stroke (width 0) (type default))
+  )
   (wire (pts (xy 49.53 52.07) (xy 59.69 52.07))
     (stroke (width 0) (type default))
@@
     (stroke (width 0) (type default))
   )
+  (wire (pts (xy 127 66.04) (xy 138.43 66.04))
+    (stroke (width 0) (type default))
+  )
   (wire (pts (xy 83.82 73.66) (xy 83.82 74.93))
     (stroke (width 0) (type default))
@@
   )
   (wire (pts (xy 49.53 29.21) (xy 66.04 29.21))
+    (stroke (width 0) (type default))
+  )
+  (wire (pts (xy 138.43 57.15) (xy 138.43 66.04))
     (stroke (width 0) (type default))
   )
@@
       (effects (font (size 1.27 1.27)))
     )
-    (property "Value" "10K" (at 105.41 66.04 90)
+    (property "Value" "1K" (at 105.41 66.04 90)
       (effects (font (size 1.27 1.27)))
     )
@@
     )
   )
+  (symbol (lib_id "Switch:SW_Push") (at 121.92 49.53 0) (unit 1)
+    (in_bom yes) (on_board yes) (dnp no) (fields_autoplaced)
+    (property "Reference" "SW1" (at 121.92 41.91 0)
+      (effects (font (size 1.27 1.27)))
+    )
+    (property "Value" "SW_Push" (at 121.92 44.45 0)
+      (effects (font (size 1.27 1.27)))
+    )
+    (property "Footprint" "" (at 121.92 44.45 0)
+      (effects (font (size 1.27 1.27)) hide)
+    )
+    (property "Datasheet" "~" (at 121.92 44.45 0)
+      (effects (font (size 1.27 1.27)) hide)
+    )
+    (pin "1")
+    (pin "2")
+    (instances
+      (project "pic10F200_servo"
+        (path "/73c37809-7617-4b9f-a70a-5c31575fa255"
+          (reference "SW1") (unit 1)
+        )
+      )
+    )
+  )
+  (symbol (lib_id "Switch:SW_Push") (at 121.92 66.04 0) (unit 1)
+    (in_bom yes) (on_board yes) (dnp no)
+    (property "Reference" "SW2" (at 121.92 68.58 0)
+      (effects (font (size 1.27 1.27)))
+    )
+    (property "Value" "SW_Push" (at 123.19 71.12 0)
+      (effects (font (size 1.27 1.27)))
+    )
+    (property "Footprint" "" (at 121.92 60.96 0)
+      (effects (font (size 1.27 1.27)) hide)
+    )
+    (property "Datasheet" "~" (at 121.92 60.96 0)
+      (effects (font (size 1.27 1.27)) hide)
+    )
+    (pin "1")
+    (pin "2")
+    (instances
+      (project "pic10F200_servo"
+        (path "/73c37809-7617-4b9f-a70a-5c31575fa255"
+          (reference "SW2") (unit 1)
+        )
+      )
+    )
+  )
   (symbol (lib_id "Motor:Motor_Servo") (at 41.91 52.07 180) (unit 1)
     (in_bom yes) (on_board yes) (dnp no) (fields_autoplaced)
@@
         (path "/73c37809-7617-4b9f-a70a-5c31575fa255"
           (reference "#PWR02") (unit 1)
+        )
+      )
+    )
+  )
+  (symbol (lib_id "power:GND") (at 138.43 57.15 90) (unit 1)
+    (in_bom yes) (on_board yes) (dnp no) (fields_autoplaced)
+    (property "Reference" "#PWR03" (at 144.78 57.15 0)
+      (effects (font (size 1.27 1.27)) hide)
+    )
+    (property "Value" "GND" (at 142.24 57.15 90)
+      (effects (font (size 1.27 1.27)) (justify right))
+    )
+    (property "Footprint" "" (at 138.43 57.15 0)
+      (effects (font (size 1.27 1.27)) hide)
+    )
+    (property "Datasheet" "" (at 138.43 57.15 0)
+      (effects (font (size 1.27 1.27)) hide)
+    )
+    (pin "1")
+    (instances
+      (project "pic10F200_servo"
+        (path "/73c37809-7617-4b9f-a70a-5c31575fa255"
+          (reference "#PWR03") (unit 1)
         )
       )
@@
       (effects (font (size 1.27 1.27)))
     )
-    (property "Value" "10K" (at 105.41 50.8 90)
-      (effects (font (size 1.27 1.27)))
-    )
+    (property "Value" "1K" (at 105.41 50.8 90)
+      (effects (font (size 1.27 1.27)))
+    )
