File: projects/16-SERVO/PIC10F200/KiCad/pic10F200_servo.kicad_sch (KiCad schematic)
At the start: 5 parts, among them M1 Motor_Servo, U1 PIC10F200-IP

Commit message: Doc
Parts:
- added SW1, SW2, SW3: SW_Push, symbol Switch:SW_Push
- R1, R2, R3: value 10K -> 2.2K
Connections:
- net +5V: no longer R1.1
- net GND: now also SW1.2, SW2.2, SW3.2
- net at R3.1: now also SW2.1
- net at R2.1: now also SW1.1
- new net: R1.1, SW3.1
Other:
- title: Basic Servo Controll with PIC16F628A -> Basic Servo Controll with PIC10F200 and 3 buttons
Changed lines of the file:
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@@
   (paper "User" 200 140.005)
   (title_block
-    (title "Basic Servo Controll with PIC16F628A")
+    (title "Basic Servo Controll with PIC10F200 and 3 buttons")
     (company "Ricardo Lima Caratti")
   )
   (junction (at 66.04 29.21) (diameter 0) (color 0 0 0 0)
   )
-  (junction (at 83.82 73.66) (diameter 0) (color 0 0 0 0)
+  (junction (at 146.05 69.85) (diameter 0) (color 0 0 0 0)
+  )
+  (junction (at 146.05 57.15) (diameter 0) (color 0 0 0 0)
   )
   (wire (pts (xy 66.04 29.21) (xy 83.82 29.21))
     (stroke (width 0) (type default))
   )
-  (wire (pts (xy 83.82 72.39) (xy 83.82 73.66))
-    (stroke (width 0) (type default))
-  )
-  (wire (pts (xy 63.5 73.66) (xy 83.82 73.66))
+  (wire (pts (xy 146.05 69.85) (xy 146.05 57.15))
+    (stroke (width 0) (type default))
+  )
+  (wire (pts (xy 63.5 85.09) (xy 119.38 85.09))
+    (stroke (width 0) (type default))
+  )
+  (wire (pts (xy 83.82 72.39) (xy 83.82 74.93))
     (stroke (width 0) (type default))
   )
@@
     (stroke (width 0) (type default))
   )
+  (wire (pts (xy 146.05 85.09) (xy 146.05 69.85))
+    (stroke (width 0) (type default))
+  )
+  (wire (pts (xy 118.11 59.69) (xy 118.11 69.85))
+    (stroke (width 0) (type default))
+  )
+  (wire (pts (xy 128.27 46.99) (xy 146.05 46.99))
+    (stroke (width 0) (type default))
+  )
   (wire (pts (xy 99.06 59.69) (xy 101.6 59.69))
     (stroke (width 0) (type default))
@@
     (stroke (width 0) (type default))
   )
+  (wire (pts (xy 128.27 69.85) (xy 146.05 69.85))
+    (stroke (width 0) (type default))
+  )
+  (wire (pts (xy 109.22 54.61) (xy 118.11 54.61))
+    (stroke (width 0) (type default))
+  )
+  (wire (pts (xy 146.05 46.99) (xy 146.05 57.15))
+    (stroke (width 0) (type default))
+  )
   (wire (pts (xy 68.58 59.69) (xy 63.5 59.69))
     (stroke (width 0) (type default))
   )
-  (wire (pts (xy 63.5 71.12) (xy 63.5 73.66))
-    (stroke (width 0) (type default))
-  )
-  (wire (pts (xy 83.82 73.66) (xy 83.82 74.93))
+  (wire (pts (xy 63.5 71.12) (xy 63.5 85.09))
+    (stroke (width 0) (type default))
+  )
+  (wire (pts (xy 109.22 59.69) (xy 118.11 59.69))
+    (stroke (width 0) (type default))
+  )
+  (wire (pts (xy 118.11 54.61) (xy 118.11 46.99))
     (stroke (width 0) (type default))
   )
@@
   (wire (pts (xy 49.53 49.53) (xy 49.53 29.21))
     (stroke (width 0) (type default))
+  )
+  (wire (pts (xy 129.54 85.09) (xy 146.05 85.09))
+    (stroke (width 0) (type default))
+  )
+  (symbol (lib_id "Switch:SW_Push") (at 123.19 69.85 0) (unit 1)
+    (in_bom yes) (on_board yes) (dnp no) (fields_autoplaced)
+    (property "Reference" "SW2" (at 123.19 62.23 0)
+      (effects (font (size 1.27 1.27)))
+    )
+    (property "Value" "SW_Push" (at 123.19 64.77 0)
+      (effects (font (size 1.27 1.27)))
+    )
+    (property "Footprint" "" (at 123.19 64.77 0)
+      (effects (font (size 1.27 1.27)) hide)
+    )
+    (property "Datasheet" "~" (at 123.19 64.77 0)
+      (effects (font (size 1.27 1.27)) hide)
+    )
+    (pin "1")
+    (pin "2")
+    (instances
+      (project "pic10F200_servo"
+        (path "/73c37809-7617-4b9f-a70a-5c31575fa255"
+          (reference "SW2") (unit 1)
+        )
+      )
+    )
+  )
+  (symbol (lib_id "power:GND") (at 146.05 57.15 90) (unit 1)
+    (in_bom yes) (on_board yes) (dnp no) (fields_autoplaced)
+    (property "Reference" "#PWR03" (at 152.4 57.15 0)
+      (effects (font (size 1.27 1.27)) hide)
+    )
+    (property "Value" "GND" (at 149.86 57.15 90)
+      (effects (font (size 1.27 1.27)) (justify right))
+    )
+    (property "Footprint" "" (at 146.05 57.15 0)
+      (effects (font (size 1.27 1.27)) hide)
+    )
+    (property "Datasheet" "" (at 146.05 57.15 0)
+      (effects (font (size 1.27 1.27)) hide)
+    )
+    (pin "1")
+    (instances
+      (project "pic10F200_servo"
+        (path "/73c37809-7617-4b9f-a70a-5c31575fa255"
+          (reference "#PWR03") (unit 1)
+        )
+      )
+    )
+  )
+  (symbol (lib_id "Switch:SW_Push") (at 123.19 46.99 0) (unit 1)
+    (in_bom yes) (on_board yes) (dnp no) (fields_autoplaced)
+    (property "Reference" "SW1" (at 123.19 39.37 0)
+      (effects (font (size 1.27 1.27)))
+    )
+    (property "Value" "SW_Push" (at 123.19 41.91 0)
+      (effects (font (size 1.27 1.27)))
+    )
+    (property "Footprint" "" (at 123.19 41.91 0)
+      (effects (font (size 1.27 1.27)) hide)
+    )
+    (property "Datasheet" "~" (at 123.19 41.91 0)
+      (effects (font (size 1.27 1.27)) hide)
+    )
+    (pin "1")
+    (pin "2")
+    (instances
+      (project "pic10F200_servo"
+        (path "/73c37809-7617-4b9f-a70a-5c31575fa255"
+          (reference "SW1") (unit 1)
+        )
+      )
+    )
   )
   (symbol (lib_id "Device:R_US") (at 105.41 59.69 270) (unit 1)
@@
       (effects (font (size 1.27 1.27)))
     )
-    (property "Value" "10K" (at 105.41 66.04 90)
+    (property "Value" "2.2K" (at 105.41 66.04 90)
       (effects (font (size 1.27 1.27)))
     )
@@
       (effects (font (size 1.27 1.27)) (justify right))
     )
-    (property "Value" "10K" (at 66.04 68.58 0)
+    (property "Value" "2.2K" (at 66.04 68.58 0)
       (effects (font (size 1.27 1.27)) (justify right))
     )
@@
         (path "/73c37809-7617-4b9f-a70a-5c31575fa255"
           (reference "#PWR02") (unit 1)
+        )
+      )
+    )
+  )
+  (symbol (lib_id "Switch:SW_Push") (at 124.46 85.09 0) (unit 1)
+    (in_bom yes) (on_board yes) (dnp no) (fields_autoplaced)
+    (property "Reference" "SW3" (at 124.46 77.47 0)
+      (effects (font (size 1.27 1.27)))
+    )
+    (property "Value" "SW_Push" (at 124.46 80.01 0)
+      (effects (font (size 1.27 1.27)))
+    )
+    (property "Footprint" "" (at 124.46 80.01 0)
+      (effects (font (size 1.27 1.27)) hide)
+    )
+    (property "Datasheet" "~" (at 124.46 80.01 0)
+      (effects (font (size 1.27 1.27)) hide)
+    )
+    (pin "1")
+    (pin "2")
+    (instances
+      (project "pic10F200_servo"
+        (path "/73c37809-7617-4b9f-a70a-5c31575fa255"
+          (reference "SW3") (unit 1)
         )
       )
@@
       (effects (font (size 1.27 1.27)))
     )
-    (property "Value" "10K" (at 105.41 50.8 90)
-      (effects (font (size 1.27 1.27)))
-    )
+    (property "Value" "2.2K" (at 105.41 50.8 90)
+      (effects (font (size 1.27 1.27)))
+    )
