File: projects/05-PWM-SPEED-COOLER/PIC12F675/KiCad/PIC12F675_pwm_lm35_4_wire_cooler.kicad_sch (KiCad schematic)
At the start: 6 parts, among them M1 Motor_DC, Q1 2N2222, U1 PIC12F675-IP, U2 LM35-LP

Commit message: Doc
Parts:
- removed M1: Motor_DC, symbol Motor:Motor_DC
- removed Q1: 2N2222, Package_TO_SOT_THT:TO-39-3, symbol Transistor_BJT:2N2219
- added M2: Fan_4pin, symbol Motor:Fan_4pin
Connections:
- net +5V: now also M2.2 (+)
- net GND: now also M2.1 (-)
- net at R2.2: now also M2.4 (PWM)
Other:
- title: PIC12F675 PWM with  Cooler and LM35 -> PIC12F675 PWM with  4-wire Cooler and LM35
- moved on the sheet: R2
Changed lines of the file:
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@@
   (paper "User" 170.002 140.005)
   (title_block
-    (title "PIC12F675 PWM with  Cooler and LM35")
+    (title "PIC12F675 PWM with  4-wire Cooler and LM35")
     (company "Ricardo Lima Caratti")
     (comment 1 "Fiver Indicator wirh LM35  and LED using the PIC12F675. ")
@@
   (junction (at 86.36 73.66) (diameter 0) (color 0 0 0 0)
   )
+  (junction (at 113.03 30.48) (diameter 0) (color 0 0 0 0)
+  )
   (wire (pts (xy 86.36 73.66) (xy 86.36 82.55))
     (stroke (width 0) (type default))
@@
     (stroke (width 0) (type default))
   )
-  (wire (pts (xy 86.36 73.66) (xy 129.54 73.66))
-    (stroke (width 0) (type default))
-  )
-  (wire (pts (xy 146.05 63.5) (xy 146.05 58.42))
-    (stroke (width 0) (type default))
-  )
-  (wire (pts (xy 101.6 68.58) (xy 107.95 68.58))
+  (wire (pts (xy 86.36 73.66) (xy 134.62 73.66))
+    (stroke (width 0) (type default))
+  )
+  (wire (pts (xy 134.62 57.15) (xy 134.62 73.66))
+    (stroke (width 0) (type default))
+  )
+  (wire (pts (xy 101.6 54.61) (xy 105.41 54.61))
     (stroke (width 0) (type default))
   )
@@
     (stroke (width 0) (type default))
   )
+  (wire (pts (xy 134.62 44.45) (xy 134.62 30.48))
+    (stroke (width 0) (type default))
+  )
+  (wire (pts (xy 134.62 30.48) (xy 113.03 30.48))
+    (stroke (width 0) (type default))
+  )
   (wire (pts (xy 113.03 30.48) (xy 86.36 30.48))
     (stroke (width 0) (type default))
   )
-  (wire (pts (xy 146.05 27.94) (xy 146.05 45.72))
-    (stroke (width 0) (type default))
-  )
-  (wire (pts (xy 129.54 63.5) (xy 146.05 63.5))
-    (stroke (width 0) (type default))
-  )
   (wire (pts (xy 62.23 49.53) (xy 71.12 49.53))
     (stroke (width 0) (type default))
   )
-  (wire (pts (xy 101.6 54.61) (xy 101.6 68.58))
-    (stroke (width 0) (type default))
-  )
   (wire (pts (xy 52.07 41.91) (xy 52.07 30.48))
     (stroke (width 0) (type default))
@@
     (stroke (width 0) (type default))
   )
-  (wire (pts (xy 115.57 68.58) (xy 121.92 68.58))
+  (wire (pts (xy 113.03 54.61) (xy 127 54.61))
     (stroke (width 0) (type default))
   )
@@
     (pin "1")
     (instances
-      (project "PIC12F675_pwm_lm35"
+      (project "PIC12F675_pwm_lm35_4_wire_cooler"
         (path "/e310d602-5c89-43bf-b83f-8bd293d0af3f"
           (reference "#PWR01") (unit 1)
+        )
+      )
+    )
+  )
+  (symbol (lib_id "Motor:Fan_4pin") (at 134.62 52.07 0) (unit 1)
+    (in_bom yes) (on_board yes) (dnp no) (fields_autoplaced)
+    (property "Reference" "M2" (at 139.7 50.8 0)
+      (effects (font (size 1.27 1.27)) (justify left))
+    )
+    (property "Value" "Fan_4pin" (at 139.7 53.34 0)
+      (effects (font (size 1.27 1.27)) (justify left))
+    )
+    (property "Footprint" "" (at 134.62 51.816 0)
+      (effects (font (size 1.27 1.27)) hide)
+    )
+    (property "Datasheet" "http://www.formfactors.org/developer%5Cspecs%5Crev1_2_public.pdf" (at 134.62 51.816 0)
+      (effects (font (size 1.27 1.27)) hide)
+    )
+    (pin "1")
+    (pin "2")
+    (pin "3")
+    (pin "4")
+    (instances
+      (project "PIC12F675_pwm_lm35_4_wire_cooler"
+        (path "/e310d602-5c89-43bf-b83f-8bd293d0af3f"
+          (reference "M2") (unit 1)
         )
       )
@@
     (pin "8")
     (instances
-      (project "PIC12F675_pwm_lm35"
+      (project "PIC12F675_pwm_lm35_4_wire_cooler"
         (path "/e310d602-5c89-43bf-b83f-8bd293d0af3f"
           (reference "U1") (unit 1)
@@
     (pin "2")
     (instances
-      (project "PIC12F675_pwm_lm35"
+      (project "PIC12F675_pwm_lm35_4_wire_cooler"
         (path "/e310d602-5c89-43bf-b83f-8bd293d0af3f"
           (reference "R1") (unit 1)
-        )
-      )
-    )
-  )
-  (symbol (lib_id "power:+5V") (at 146.05 27.94 0) (unit 1)
-    (in_bom yes) (on_board yes) (dnp no) (fields_autoplaced)
-    (property "Reference" "#PWR04" (at 146.05 31.75 0)
-      (effects (font (size 1.27 1.27)) hide)
-    )
-    (property "Value" "+5V" (at 146.05 22.86 0)
-      (effects (font (size 1.27 1.27)))
-    )
-    (property "Footprint" "" (at 146.05 27.94 0)
-      (effects (font (size 1.27 1.27)) hide)
-    )
-    (property "Datasheet" "" (at 146.05 27.94 0)
-      (effects (font (size 1.27 1.27)) hide)
-    )
-    (pin "1")
-    (instances
-      (project "PIC12F675_pwm_lm35"
-        (path "/e310d602-5c89-43bf-b83f-8bd293d0af3f"
-          (reference "#PWR04") (unit 1)
-        )
-      )
-    )
-  )
-  (symbol (lib_id "Motor:Motor_DC") (at 146.05 50.8 0) (unit 1)
-    (in_bom yes) (on_board yes) (dnp no) (fields_autoplaced)
-    (property "Reference" "M1" (at 151.13 52.07 0)
-      (effects (font (size 1.27 1.27)) (justify left))
-    )
-    (property "Value" "Motor_DC" (at 151.13 54.61 0)
-      (effects (font (size 1.27 1.27)) (justify left))
-    )
-    (property "Footprint" "" (at 146.05 53.086 0)
-      (effects (font (size 1.27 1.27)) hide)
-    )
-    (property "Datasheet" "~" (at 146.05 53.086 0)
-      (effects (font (size 1.27 1.27)) hide)
-    )
-    (pin "1")
-    (pin "2")
-    (instances
-      (project "PIC12F675_pwm_lm35"
-        (path "/e310d602-5c89-43bf-b83f-8bd293d0af3f"
-          (reference "M1") (unit 1)
         )
       )
@@
     (pin "3")
     (instances
-      (project "PIC12F675_pwm_lm35"
+      (project "PIC12F675_pwm_lm35_4_wire_cooler"
         (path "/e310d602-5c89-43bf-b83f-8bd293d0af3f"
           (reference "U2") (unit 1)
@@
     )
   )
-  (symbol (lib_id "Device:R") (at 111.76 68.58 90) (unit 1)
-    (in_bom yes) (on_board yes) (dnp no) (fields_autoplaced)
-    (property "Reference" "R2" (at 111.76 62.23 90)
-      (effects (font (size 1.27 1.27)))
-    )
-    (property "Value" "1K" (at 111.76 64.77 90)
-      (effects (font (size 1.27 1.27)))
-    )
-    (property "Footprint" "" (at 111.76 70.358 90)
-      (effects (font (size 1.27 1.27)) hide)
-    )
-    (property "Datasheet" "~" (at 111.76 68.58 0)
-      (effects (font (size 1.27 1.27)) hide)
-    )
-    (pin "1")
-    (pin "2")
-    (instances
-      (project "PIC12F675_pwm_lm35"
+  (symbol (lib_id "Device:R") (at 109.22 54.61 90) (unit 1)
+    (in_bom yes) (on_board yes) (dnp no)
+    (property "Reference" "R2" (at 107.95 57.15 90)
+      (effects (font (size 1.27 1.27)))
+    )
+    (property "Value" "1K" (at 107.95 59.69 90)
+      (effects (font (size 1.27 1.27)))
+    )
+    (property "Footprint" "" (at 109.22 56.388 90)
+      (effects (font (size 1.27 1.27)) hide)
+    )
+    (property "Datasheet" "~" (at 109.22 54.61 0)
+      (effects (font (size 1.27 1.27)) hide)
+    )
+    (pin "1")
+    (pin "2")
+    (instances
+      (project "PIC12F675_pwm_lm35_4_wire_cooler"
         (path "/e310d602-5c89-43bf-b83f-8bd293d0af3f"
           (reference "R2") (unit 1)
@@
     (pin "1")
     (instances
-      (project "PIC12F675_pwm_lm35"
+      (project "PIC12F675_pwm_lm35_4_wire_cooler"
         (path "/e310d602-5c89-43bf-b83f-8bd293d0af3f"
           (reference "#PWR02") (unit 1)
         )
       )
-    )
-  )
-  (symbol (lib_id "Transistor_BJT:2N2219") (at 127 68.58 0) (mirror x) (unit 1)
-    (in_bom yes) (on_board yes) (dnp no)
-    (property "Reference" "Q1" (at 132.08 69.85 0)
-      (effects (font (size 1.27 1.27)) (justify left))
-    )
-    (property "Value" "2N2222" (at 132.08 67.31 0)
-      (effects (font (size 1.27 1.27)) (justify left))
-    )
-    (property "Footprint" "Package_TO_SOT_THT:TO-39-3" (at 132.08 66.675 0)
-      (effects (font (size 1.27 1.27) italic) (justify left) hide)
-    )
-    (property "Datasheet" "http://www.onsemi.com/pub_link/Collateral/2N2219-D.PDF" (at 127 68.58 0)
-      (effects (font (size 1.27 1.27)) (justify left) hide)
-    )
-    (pin "1")
-    (pin "2")
-    (pin "3")
-    (instances
-      (project "PIC12F675_pwm_lm35"
-        (path "/e310d602-5c89-43bf-b83f-8bd293d0af3f"
-          (reference "Q1") (unit 1)
-        )
-      )
