File: projects/05-PWM-SPEED-COOLER/PIC12F675/KiCad/pic12F675_pwm.kicad_sch (KiCad schematic)
At the start: 2 parts, among them U1 PIC12F675-IP

Commit message: Doc
Parts:
- added M1: Motor_DC, symbol Motor:Motor_DC
- added R1: 1K, symbol Device:R
- added U2: L293D, Package_DIP:DIP-16_W7.62mm, symbol Driver_Motor:L293D
Connections:
- net +5V: now also U2.1 (EN1,2), U2.16 (VCC1)
- net GND: now also M1.2 (-), U2.12 (GND), U2.13 (GND), U2.4 (GND), U2.5 (GND)
- net at U1.2 (GP5): now also R1.1
- new net: M1.1 (+), U2.3 (1Y)
- new net: R1.2, U2.2 (1A)
- new net +12V: U2.8 (VCC2)
Other:
- title: Basic PWM with PIC12F675, ADC, Timer and Interrupt -> PIC12F675 with  H-bridge L293D - ADC, Timer and Interrupt
