File: projects/16-SERVO/PIC12F675/KiCad/pic12F675_pwm_servo.kicad_sch (KiCad schematic)
At the start: 3 parts, among them M1 Motor_Servo, U1 PIC12F675-IP

Commit message: Doc
Parts:
- added R1: 1K, symbol Device:R
Connections:
- net at U1.2 (GP5): now also R1.2; no longer M1.1 (PWM)
- new net: M1.1 (PWM), R1.1
Changed lines of the file:
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@@
     (stroke (width 0) (type default))
   )
-  (wire (pts (xy 62.23 49.53) (xy 83.82 49.53))
+  (wire (pts (xy 78.74 49.53) (xy 83.82 49.53))
     (stroke (width 0) (type default))
   )
@@
   )
   (wire (pts (xy 99.06 33.02) (xy 99.06 36.83))
+    (stroke (width 0) (type default))
+  )
+  (wire (pts (xy 62.23 49.53) (xy 71.12 49.53))
     (stroke (width 0) (type default))
   )
@@
         )
       )
+    )
+  )
+  (symbol (lib_id "Device:R") (at 74.93 49.53 90) (unit 1)
+    (in_bom yes) (on_board yes) (dnp no) (fields_autoplaced)
+    (property "Reference" "R1" (at 74.93 43.18 90)
+      (effects (font (size 1.27 1.27)))
+    )
+    (property "Value" "1K" (at 74.93 45.72 90)
+      (effects (font (size 1.27 1.27)))
+    )
+    (property "Footprint" "" (at 74.93 51.308 90)
+      (effects (font (size 1.27 1.27)) hide)
+    )
+    (property "Datasheet" "~" (at 74.93 49.53 0)
+      (effects (font (size 1.27 1.27)) hide)
+    )
+    (pin "1")
+    (pin "2")
+    (instances
+      (project "pic12F675_pwm_servo"
+        (path "/73c37809-7617-4b9f-a70a-5c31575fa255"
+          (reference "R1") (unit 1)
+        )
+      )

Commit message: Doc
Parts:
- added R2: 10K, symbol Device:R
Connections:
- net +5V: now also R2.1
- net at U1.4 (GP3): now also R2.2
Changed lines of the file:
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@@
     (company "Ricardo Lima Caratti")
+  )
+  (junction (at 83.82 71.12) (diameter 0) (color 0 0 0 0)
   )
   (junction (at 123.19 55.88) (diameter 0) (color 0 0 0 0)
@@
   (junction (at 99.06 33.02) (diameter 0) (color 0 0 0 0)
   )
+  (wire (pts (xy 83.82 71.12) (xy 99.06 71.12))
+    (stroke (width 0) (type default))
+  )
   (wire (pts (xy 114.3 55.88) (xy 123.19 55.88))
     (stroke (width 0) (type default))
   )
-  (wire (pts (xy 67.31 71.12) (xy 99.06 71.12))
+  (wire (pts (xy 83.82 67.31) (xy 83.82 71.12))
+    (stroke (width 0) (type default))
+  )
+  (wire (pts (xy 67.31 71.12) (xy 83.82 71.12))
     (stroke (width 0) (type default))
   )
@@
   )
   (wire (pts (xy 99.06 67.31) (xy 99.06 71.12))
+    (stroke (width 0) (type default))
+  )
+  (wire (pts (xy 83.82 54.61) (xy 83.82 59.69))
     (stroke (width 0) (type default))
   )
@@
         )
       )
+    )
+  )
+  (symbol (lib_id "Device:R") (at 83.82 63.5 180) (unit 1)
+    (in_bom yes) (on_board yes) (dnp no)
+    (property "Reference" "R2" (at 77.47 62.23 0)
+      (effects (font (size 1.27 1.27)) (justify right))
+    )
+    (property "Value" "10K" (at 77.47 64.77 0)
+      (effects (font (size 1.27 1.27)) (justify right))
+    )
+    (property "Footprint" "" (at 85.598 63.5 90)
+      (effects (font (size 1.27 1.27)) hide)
+    )
+    (property "Datasheet" "~" (at 83.82 63.5 0)
+      (effects (font (size 1.27 1.27)) hide)
+    )
+    (pin "1")
+    (pin "2")
+    (instances
+      (project "pic12F675_pwm_servo"
+        (path "/73c37809-7617-4b9f-a70a-5c31575fa255"
+          (reference "R2") (unit 1)
+        )
+      )
