File: projects/18-PUSH_BUTTON_INTERRUPT/PIC12F675/KiCad/PIC12F675_PUSH_BUTTON_INTERRUPT.kicad_sch (KiCad schematic)
At the start: 6 parts, among them SW1 SW_Push, U1 PIC12F675-IP

Commit message: Doc
Connections:
- net at U1.5 (GP2): now also R2.2
- net at U1.7 (GP0): no longer R2.2
Other:
- moved on the sheet: R2, SW1
Changed lines of the file:
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@@
   (junction (at 80.01 69.85) (diameter 0) (color 0 0 0 0)
   )
-  (wire (pts (xy 52.07 45.72) (xy 53.34 45.72))
-    (stroke (width 0) (type default))
-  )
-  (wire (pts (xy 41.91 45.72) (xy 41.91 69.85))
+  (wire (pts (xy 52.07 50.8) (xy 53.34 50.8))
+    (stroke (width 0) (type default))
+  )
+  (wire (pts (xy 41.91 50.8) (xy 41.91 69.85))
     (stroke (width 0) (type default))
   )
@@
     (stroke (width 0) (type default))
   )
+  (wire (pts (xy 60.96 50.8) (xy 64.77 50.8))
+    (stroke (width 0) (type default))
+  )
   (wire (pts (xy 95.25 50.8) (xy 95.25 62.23))
     (stroke (width 0) (type default))
@@
     (stroke (width 0) (type default))
   )
-  (wire (pts (xy 60.96 45.72) (xy 64.77 45.72))
-    (stroke (width 0) (type default))
-  )
   (wire (pts (xy 95.25 62.23) (xy 100.33 62.23))
     (stroke (width 0) (type default))
@@
     )
   )
-  (symbol (lib_id "Switch:SW_Push") (at 46.99 45.72 0) (unit 1)
-    (in_bom yes) (on_board yes) (dnp no) (fields_autoplaced)
-    (property "Reference" "SW1" (at 46.99 38.1 0)
-      (effects (font (size 1.27 1.27)))
-    )
-    (property "Value" "SW_Push" (at 46.99 40.64 0)
-      (effects (font (size 1.27 1.27)))
-    )
-    (property "Footprint" "" (at 46.99 40.64 0)
-      (effects (font (size 1.27 1.27)) hide)
-    )
-    (property "Datasheet" "~" (at 46.99 40.64 0)
+  (symbol (lib_id "Switch:SW_Push") (at 46.99 50.8 0) (unit 1)
+    (in_bom yes) (on_board yes) (dnp no) (fields_autoplaced)
+    (property "Reference" "SW1" (at 46.99 43.18 0)
+      (effects (font (size 1.27 1.27)))
+    )
+    (property "Value" "SW_Push" (at 46.99 45.72 0)
+      (effects (font (size 1.27 1.27)))
+    )
+    (property "Footprint" "" (at 46.99 45.72 0)
+      (effects (font (size 1.27 1.27)) hide)
+    )
+    (property "Datasheet" "~" (at 46.99 45.72 0)
       (effects (font (size 1.27 1.27)) hide)
     )
@@
     )
   )
-  (symbol (lib_id "Device:R") (at 57.15 45.72 90) (unit 1)
-    (in_bom yes) (on_board yes) (dnp no) (fields_autoplaced)
-    (property "Reference" "R2" (at 57.15 39.37 90)
-      (effects (font (size 1.27 1.27)))
-    )
-    (property "Value" "1K" (at 57.15 41.91 90)
-      (effects (font (size 1.27 1.27)))
-    )
-    (property "Footprint" "" (at 57.15 47.498 90)
-      (effects (font (size 1.27 1.27)) hide)
-    )
-    (property "Datasheet" "~" (at 57.15 45.72 0)
-      (effects (font (size 1.27 1.27)) hide)
-    )
+  (symbol (lib_id "Device:R") (at 57.15 50.8 90) (unit 1)
+    (in_bom yes) (on_board yes) (dnp no) (fields_autoplaced)
+    (property "Reference" "R2" (at 57.15 44.45 90)
+      (effects (font (size 1.27 1.27)))
+    )
+    (property "Value" "1K" (at 57.15 46.99 90)
+      (effects (font (size 1.27 1.27)))
+    )
+    (property "Footprint" "" (at 57.15 52.578 90)
+      (effects (font (size 1.27 1.27)) hide)
+    )
+    (property "Datasheet" "~" (at 57.15 50.8 0)
+      (effects (font (size 1.27 1.27)) hide)
+    )

Commit message: Doc
Parts:
- added C1: 22nF, symbol Device:C
Connections:
- net GND: now also C1.2
- net at R2.1, SW1.2: now also C1.1
Other:
- note added: "Debounce Capacitor"
Changed lines of the file:
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@@
   (junction (at 80.01 69.85) (diameter 0) (color 0 0 0 0)
   )
+  (junction (at 52.07 69.85) (diameter 0) (color 0 0 0 0)
+  )
+  (junction (at 52.07 50.8) (diameter 0) (color 0 0 0 0)
+  )
   (wire (pts (xy 52.07 50.8) (xy 53.34 50.8))
     (stroke (width 0) (type default))
@@
     (stroke (width 0) (type default))
   )
+  (wire (pts (xy 52.07 63.5) (xy 52.07 69.85))
+    (stroke (width 0) (type default))
+  )
   (wire (pts (xy 119.38 62.23) (xy 119.38 69.85))
     (stroke (width 0) (type default))
   )
+  (wire (pts (xy 52.07 50.8) (xy 52.07 55.88))
+    (stroke (width 0) (type default))
+  )
   (wire (pts (xy 60.96 50.8) (xy 64.77 50.8))
     (stroke (width 0) (type default))
@@
     (stroke (width 0) (type default))
   )
-  (wire (pts (xy 41.91 69.85) (xy 80.01 69.85))
+  (wire (pts (xy 41.91 69.85) (xy 52.07 69.85))
     (stroke (width 0) (type default))
   )
@@
   (wire (pts (xy 80.01 20.32) (xy 80.01 33.02))
     (stroke (width 0) (type default))
+  )
+  (wire (pts (xy 52.07 69.85) (xy 80.01 69.85))
+    (stroke (width 0) (type default))
+  )
+  (text "Debounce\nCapacitor" (at 54.61 66.04 0)
+    (effects (font (size 1.27 1.27)) (justify left bottom))
   )
   (symbol (lib_id "power:+5V") (at 80.01 20.32 0) (unit 1)
@@
         )
       )
+    )
+  )
+  (symbol (lib_id "Device:C") (at 52.07 59.69 0) (unit 1)
+    (in_bom yes) (on_board yes) (dnp no) (fields_autoplaced)
+    (property "Reference" "C1" (at 55.88 58.42 0)
+      (effects (font (size 1.27 1.27)) (justify left))
+    )
+    (property "Value" "22nF" (at 55.88 60.96 0)
+      (effects (font (size 1.27 1.27)) (justify left))
+    )
+    (property "Footprint" "" (at 53.0352 63.5 0)
+      (effects (font (size 1.27 1.27)) hide)
+    )
+    (property "Datasheet" "~" (at 52.07 59.69 0)
+      (effects (font (size 1.27 1.27)) hide)
+    )
+    (pin "1")
+    (pin "2")
+    (instances
+      (project "PIC12F675_PUSH_BUTTON_INTERRUPT"
+        (path "/e310d602-5c89-43bf-b83f-8bd293d0af3f"
+          (reference "C1") (unit 1)
+        )
+      )
