File: projects/18-PUSH_BUTTON_INTERRUPT/PIC16F628A/KiCad/PIC16F628A_PUSH_BUTTON_INTERRUPT.kicad_sch (KiCad schematic)
At the start: 6 parts, among them SW1 SW_Push, U1 PIC16F628A-IP

Commit message: DOC
Connections:
- net at R3.1: now also D1.2 (A); no longer U1.17 (AN0/RA0)
- net at R3.2: now also U1.9 (RB3/CCP1); no longer D1.2 (A)
Changed lines of the file:
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@@
     (comment 1 "A minimalist project with PIC16F628A, push button and interrupt. ")
   )
+  (junction (at 41.91 72.39) (diameter 0) (color 0 0 0 0)
+  )
   (junction (at 90.17 72.39) (diameter 0) (color 0 0 0 0)
   )
-  (wire (pts (xy 30.48 72.39) (xy 90.17 72.39))
-    (stroke (width 0) (type default))
-  )
-  (wire (pts (xy 118.11 40.64) (xy 121.92 40.64))
+  (wire (pts (xy 30.48 72.39) (xy 41.91 72.39))
     (stroke (width 0) (type default))
   )
@@
     (stroke (width 0) (type default))
   )
-  (wire (pts (xy 129.54 40.64) (xy 133.35 40.64))
-    (stroke (width 0) (type default))
-  )
-  (wire (pts (xy 140.97 40.64) (xy 140.97 72.39))
+  (wire (pts (xy 41.91 60.96) (xy 41.91 72.39))
+    (stroke (width 0) (type default))
+  )
+  (wire (pts (xy 48.26 48.26) (xy 41.91 48.26))
     (stroke (width 0) (type default))
   )
@@
     (stroke (width 0) (type default))
   )
-  (wire (pts (xy 140.97 72.39) (xy 90.17 72.39))
+  (wire (pts (xy 55.88 48.26) (xy 62.23 48.26))
     (stroke (width 0) (type default))
   )
@@
     (stroke (width 0) (type default))
   )
+  (wire (pts (xy 41.91 48.26) (xy 41.91 53.34))
+    (stroke (width 0) (type default))
+  )
+  (wire (pts (xy 41.91 72.39) (xy 90.17 72.39))
+    (stroke (width 0) (type default))
+  )
   (symbol (lib_id "Switch:SW_Push") (at 39.37 40.64 0) (unit 1)
     (in_bom yes) (on_board yes) (dnp no) (fields_autoplaced)
@@
     )
   )
+  (symbol (lib_id "Device:LED") (at 41.91 57.15 90) (unit 1)
+    (in_bom yes) (on_board yes) (dnp no) (fields_autoplaced)
+    (property "Reference" "D1" (at 45.72 57.4675 90)
+      (effects (font (size 1.27 1.27)) (justify right))
+    )
+    (property "Value" "LED" (at 45.72 60.0075 90)
+      (effects (font (size 1.27 1.27)) (justify right))
+    )
+    (property "Footprint" "" (at 41.91 57.15 0)
+      (effects (font (size 1.27 1.27)) hide)
+    )
+    (property "Datasheet" "~" (at 41.91 57.15 0)
+      (effects (font (size 1.27 1.27)) hide)
+    )
+    (pin "1")
+    (pin "2")
+    (instances
+      (project "PIC16F628A_PUSH_BUTTON_INTERRUPT"
+        (path "/e310d602-5c89-43bf-b83f-8bd293d0af3f"
+          (reference "D1") (unit 1)
+        )
+      )
+    )
+  )
   (symbol (lib_id "Device:R") (at 127 53.34 90) (unit 1)
     (in_bom yes) (on_board yes) (dnp no) (fields_autoplaced)
@@
     )
   )
+  (symbol (lib_id "Device:R") (at 52.07 48.26 90) (unit 1)
+    (in_bom yes) (on_board yes) (dnp no)
+    (property "Reference" "R3" (at 52.07 50.8 90)
+      (effects (font (size 1.27 1.27)))
+    )
+    (property "Value" "1K" (at 52.07 53.34 90)
+      (effects (font (size 1.27 1.27)))
+    )
+    (property "Footprint" "" (at 52.07 50.038 90)
+      (effects (font (size 1.27 1.27)) hide)
+    )
+    (property "Datasheet" "~" (at 52.07 48.26 0)
+      (effects (font (size 1.27 1.27)) hide)
+    )
+    (pin "1")
+    (pin "2")
+    (instances
+      (project "PIC16F628A_PUSH_BUTTON_INTERRUPT"
+        (path "/e310d602-5c89-43bf-b83f-8bd293d0af3f"
+          (reference "R3") (unit 1)
+        )
+      )
+    )
+  )
   (symbol (lib_id "Device:R") (at 52.07 40.64 90) (unit 1)
     (in_bom yes) (on_board yes) (dnp no) (fields_autoplaced)
@@
         )
       )
-    )
-  )
-  (symbol (lib_id "Device:R") (at 125.73 40.64 90) (unit 1)
-    (in_bom yes) (on_board yes) (dnp no) (fields_autoplaced)
-    (property "Reference" "R3" (at 125.73 34.29 90)
-      (effects (font (size 1.27 1.27)))
-    )
-    (property "Value" "1K" (at 125.73 36.83 90)
-      (effects (font (size 1.27 1.27)))
-    )
-    (property "Footprint" "" (at 125.73 42.418 90)
-      (effects (font (size 1.27 1.27)) hide)
-    )
-    (property "Datasheet" "~" (at 125.73 40.64 0)
-      (effects (font (size 1.27 1.27)) hide)
-    )
-    (pin "1")
-    (pin "2")
-    (instances
-      (project "PIC16F628A_PUSH_BUTTON_INTERRUPT"
-        (path "/e310d602-5c89-43bf-b83f-8bd293d0af3f"
-          (reference "R3") (unit 1)
-        )
-      )
-    )
-  )
-  (symbol (lib_id "Device:LED") (at 137.16 40.64 180) (unit 1)
-    (in_bom yes) (on_board yes) (dnp no) (fields_autoplaced)
-    (property "Reference" "D1" (at 138.7475 33.02 0)
-      (effects (font (size 1.27 1.27)))
-    )
-    (property "Value" "LED" (at 138.7475 35.56 0)
-      (effects (font (size 1.27 1.27)))
-    )
-    (property "Footprint" "" (at 137.16 40.64 0)
-      (effects (font (size 1.27 1.27)) hide)
-    )
-    (property "Datasheet" "~" (at 137.16 40.64 0)
-      (effects (font (size 1.27 1.27)) hide)
-    )
-    (pin "1")
-    (pin "2")
-    (instances
-      (project "PIC16F628A_PUSH_BUTTON_INTERRUPT"
-        (path "/e310d602-5c89-43bf-b83f-8bd293d0af3f"
-          (reference "D1") (unit 1)
-        )
-      )

Commit message: Doc
Parts:
- added C1: 22nF, symbol Device:C
Connections:
- net GND: now also U1.5 (VSS), C1.2
- net at R2.1, SW1.2: now also C1.1
Other:
- note added: "Debounce Capacitor"
- moved on the sheet: D1, R1, R2, SW1, U1
