File: projects/19-74HC151_MULTIPLEXER/PIC10F220/KiCad/pic12F675_74HC151_MULTIPLEXER_SENSORS.kicad_sch (KiCad schematic)
At the start: 10 parts, among them U1 PIC12F675-IP, U3 MQ-2

Commit message: Doc
Parts:
- removed D1, D2, D3: LED, symbol Device:LED
- removed R2: 10K, symbol Device:R_US
- removed R3, R4, R5: 360R, symbol Device:R_US
- removed U3: MQ-2, Sensor:MQ-6, symbol Sensor_Gas:MQ-6
- added U2: 74151, symbol 74xx_IEEE:74151
- added U3: LM35-LP, Package_TO_SOT_THT:TO-92_Inline, symbol Sensor_Temperature:LM35-LP
Connections:
- net +5P: now also U2.16 (VCC), U3.1 (+V_{S})
- net GND: now also U2.8 (GND), U2.9 (S2), U3.3 (GND)
- net at U1.7 (GP0): now also U2.5 (Q)
- net at U1.5 (GP2): now also U2.10 (S1)
- net at U1.6 (GP1): now also U2.11 (S0)
Other:
- note removed: "A0"
- note removed: "D0"
- note removed: "GND"
- note removed: "VCC"
- moved on the sheet: R1, U1

Commit message: Doc
Parts:
- added MK1: Microphone, symbol Device:Microphone
- added R2: LDR07, OptoDevice:R_LDR_5.1x4.3mm_P3.4mm_Vertical, symbol Sensor_Optical:LDR07
- added R3: 10K, symbol Device:R_US
- added U4: A1369xUA-10, Sensor_Current:Allegro_SIP-3, symbol Sensor_Current:A1369xUA-10
Connections:
- net +5P: now also R2.1, U4.1 (VCC)
- net GND: now also MK1.1 (-), R3.2, U4.2 (GND)
- net at U2.1 (I3): now also U4.3 (VOUT)
- net at U2.2 (I2): now also R2.2, R3.1
- net at U2.3 (I1): now also MK1.2 (+)
- net at U2.4 (I0): now also U3.2 (V_{OUT})
Other:
- note added: "Sensor 1"
- note added: "Sensor 2"
- note added: "Sensor 3"
- note added: "Sensor 4"
- moved on the sheet: R1, U1, U2, U3

Commit message: Doc
Parts:
- added M1: Motor_DC, symbol Motor:Motor_DC
- added PE1: PeltierElement, symbol Device:PeltierElement
- added Q1, Q2: NMOS, symbol Simulation_SPICE:NMOS
- added R4, R5: 1K, symbol Device:R_US
Connections:
- net GND: now also Q1.3 (S), Q2.3 (S)
- net at U1.2 (GP5): now also R4.2
- net at U1.3 (GP4): now also R5.2
- new net: PE1.2, Q2.1 (D)
- new net: Q2.2 (G), R5.1
- new net: M1.2 (-), Q1.1 (D)
- new net: Q1.2 (G), R4.1
- new net +12V: M1.1 (+), PE1.1
Other:
- title: PIC12F675 with MQ-2 GAS SENSOR  and LED -> PIC10F220 and 74HC151 monitoring 4 sensors

Commit message: Doc
Parts:
- removed MK1: Microphone, symbol Device:Microphone
- removed PE1: PeltierElement, symbol Device:PeltierElement
- removed R2: LDR07, OptoDevice:R_LDR_5.1x4.3mm_P3.4mm_Vertical, symbol Sensor_Optical:LDR07
- removed R3: 10K, symbol Device:R_US
- added M2: Motor_DC, symbol Motor:Motor_DC
- added U5: LM35-LP, Package_TO_SOT_THT:TO-92_Inline, symbol Sensor_Temperature:LM35-LP
- added U6: A1369xUA-10, Sensor_Current:Allegro_SIP-3, symbol Sensor_Current:A1369xUA-10
Connections:
- net +12V: now also M2.1 (+)
- net +5P: now also U5.1 (+V_{S}), U6.1 (VCC)
- net GND: now also U5.3 (GND), U6.2 (GND)
- net at U2.2 (I2): now also U5.2 (V_{OUT})
- net at U2.3 (I1): now also U6.3 (VOUT)
- net at Q2.1 (D): now also M2.2 (-)
Other:
- note removed: "Sensor 2"
- note removed: "Sensor 3"
- moved on the sheet: U3, U4

Commit message: Doc
Other:
- note added: "Sensor 2"
- note added: "Sensor 3"
Changed lines of the file:
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@@
     (effects (font (size 1.27 1.27)) (justify left bottom))
   )
-  (text "Sensor 1" (at 16.51 93.98 0)
+  (text "Sensor 3" (at 16.51 93.98 0)
     (effects (font (size 1.27 1.27)) (justify left bottom))
   )
-  (text "Sensor 4" (at 13.97 62.23 0)
+  (text "Sensor 2" (at 15.24 63.5 0)
     (effects (font (size 1.27 1.27)) (justify left bottom))
   )

Commit message: Doc
Other:
- note added: "Y"
- note added: "__"
Changed lines of the file:
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@@
+    (effects (font (size 1.27 1.27)) (justify left bottom))
+  )
+  (text "__" (at 110.49 87.63 0)
+    (effects (font (size 1.27 1.27)) (justify left bottom))
+  )
+  (text "Y" (at 110.49 54.61 0)
     (effects (font (size 1.27 1.27)) (justify left bottom))
   )
@@
     (effects (font (size 1.27 1.27)) (justify left bottom))
   )
+  (text "Y" (at 110.49 90.17 0)
+    (effects (font (size 1.27 1.27)) (justify left bottom))
+  )

Commit message: Doc
Parts:
- removed M2: Motor_DC, symbol Motor:Motor_DC
- removed Q2: NMOS, symbol Simulation_SPICE:NMOS
- removed R5: 1K, symbol Device:R_US
- removed U1: PIC12F675-IP, Package_DIP:DIP-8_W7.62mm, symbol MCU_Microchip_PIC12:PIC12F675-IP
- removed U4: A1369xUA-10, Sensor_Current:Allegro_SIP-3, symbol Sensor_Current:A1369xUA-10
- removed U5: LM35-LP, Package_TO_SOT_THT:TO-92_Inline, symbol Sensor_Temperature:LM35-LP
- added U1: PIC10F220-IP, Package_DIP:DIP-8_W7.62mm, symbol MCU_Microchip_PIC10:PIC10F220-IP
Connections:
- net +5P: now also U1.2 (VDD)
- net GND: now also U2.10 (S1), U2.7 (~{E}), U1.7 (VSS); no longer Q1.3 (S)
- net at R1.1: now also U1.8 (GP3)
- net at U2.11 (S0): now also U1.4 (GP1)
- net at U2.5 (Q): now also U1.5 (GP0)
- net at R4.2: now also U1.3 (GP2)
Other:
- note removed: "Sensor 3"
- note removed: "Sensor 4"
- title: PIC10F220 and 74HC151 monitoring 4 sensors -> PIC10F220 and 74HC151 monitoring 2 sensors
- moved on the sheet: M1, Q1, R1, R4, U3, U6
