File: projects/19-74HC151_MULTIPLEXER/PIC12F675/KiCad/pic12F675_74HC151_MULTIPLEXER_SENSORS_V1.kicad_sch (KiCad schematic)
At the start: 11 parts, among them U1 PIC12F675-IP, U2 74151, U3 ZMCT103C, U4 ZMCT103C, U5 ZMCT103C, U6 ZMCT103C

Commit message: Doc
Parts:
- removed LS1: Speaker, symbol Device:Speaker
- removed R2: 1K, symbol Device:R_US
Other:
- note added: "This LED will flash indicating the current sensor has detected the fault."
- moved on the sheet: D1, R1, R3, U3, U4, U5, U6
