File: projects/19-74HC151_MULTIPLEXER/PIC12F675/KiCad/pic12F675_74HC151_MULTIPLEXER_SENSORS_V2.kicad_sch (KiCad schematic)
At the start: 9 parts, among them U1 PIC12F675-IP, U2 74151, U3 ZMCT103C, U4 ZMCT103C, U5 ZMCT103C, U6 ZMCT103C

Commit message: Doc
Parts:
- added U7, U8, U9: ZMCT103C, Sensor_Current:Allegro_SIP-4, symbol Sensor_Current:A1363xKTTN-1
Connections:
- net +5P: now also U7.1 (VCC), U8.1 (VCC), U9.1 (VCC)
- net GND: now also U7.4 (GND), U8.4 (GND), U9.4 (GND)
- net at U4.2 (VOUT): now also U2.3 (I1)
- net at U2.13 (I6): now also U9.2 (VOUT)
- net at U2.14 (I5): now also U8.2 (VOUT)
- net at U2.15 (I4): now also U7.2 (VOUT)
- net at U2.5 (Q): now also U1.2 (GP5)
- net at U2.6 (~{Q}): no longer U1.2 (GP5)
Other:
- note added: "Sensor 5"
- note added: "Sensor 6"
- note added: "Sensor 7"

Commit message: Doc
Connections:
- net at U1.3 (GP4): now also R3.1
Other:
- moved on the sheet: D1, R1, R3
Changed lines of the file:
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@@
     (company "Ricardo Lima Caratti")
   )
-  (junction (at 151.13 34.29) (diameter 0) (color 0 0 0 0)
+  (junction (at 151.13 38.1) (diameter 0) (color 0 0 0 0)
+  )
+  (wire (pts (xy 166.37 55.88) (xy 181.61 55.88))
+    (stroke (width 0) (type default))
+  )
+  (wire (pts (xy 181.61 55.88) (xy 181.61 62.23))
+    (stroke (width 0) (type default))
   )
   (wire (pts (xy 22.86 67.31) (xy 41.91 67.31))
@@
     (stroke (width 0) (type default))
   )
-  (wire (pts (xy 190.5 88.9) (xy 190.5 95.25))
+  (wire (pts (xy 181.61 78.74) (xy 181.61 82.55))
     (stroke (width 0) (type default))
   )
@@
     (stroke (width 0) (type default))
   )
-  (wire (pts (xy 160.02 55.88) (xy 190.5 55.88))
-    (stroke (width 0) (type default))
-  )
   (wire (pts (xy 50.8 170.18) (xy 72.39 170.18))
     (stroke (width 0) (type default))
@@
     (stroke (width 0) (type default))
   )
+  (wire (pts (xy 151.13 38.1) (xy 151.13 40.64))
+    (stroke (width 0) (type default))
+  )
   (wire (pts (xy 135.89 53.34) (xy 135.89 25.4))
     (stroke (width 0) (type default))
@@
     (stroke (width 0) (type default))
   )
-  (wire (pts (xy 191.77 34.29) (xy 151.13 34.29))
+  (wire (pts (xy 151.13 34.29) (xy 151.13 38.1))
+    (stroke (width 0) (type default))
+  )
+  (wire (pts (xy 181.61 38.1) (xy 151.13 38.1))
     (stroke (width 0) (type default))
   )
@@
     (stroke (width 0) (type default))
   )
-  (wire (pts (xy 151.13 34.29) (xy 151.13 40.64))
-    (stroke (width 0) (type default))
-  )
   (wire (pts (xy 40.64 161.29) (xy 40.64 162.56))
     (stroke (width 0) (type default))
@@
     (stroke (width 0) (type default))
   )
-  (wire (pts (xy 151.13 31.75) (xy 151.13 34.29))
-    (stroke (width 0) (type default))
-  )
   (wire (pts (xy 77.47 177.8) (xy 77.47 156.21))
     (stroke (width 0) (type default))
@@
     (stroke (width 0) (type default))
   )
-  (wire (pts (xy 151.13 71.12) (xy 151.13 76.2))
+  (wire (pts (xy 151.13 71.12) (xy 151.13 72.39))
     (stroke (width 0) (type default))
   )
@@
     (stroke (width 0) (type default))
   )
-  (wire (pts (xy 166.37 53.34) (xy 177.8 53.34))
+  (wire (pts (xy 166.37 53.34) (xy 170.18 53.34))
     (stroke (width 0) (type default))
   )
@@
     (stroke (width 0) (type default))
   )
-  (wire (pts (xy 185.42 53.34) (xy 191.77 53.34))
-    (stroke (width 0) (type default))
-  )
-  (wire (pts (xy 191.77 53.34) (xy 191.77 34.29))
+  (wire (pts (xy 177.8 53.34) (xy 181.61 53.34))
+    (stroke (width 0) (type default))
+  )
+  (wire (pts (xy 181.61 53.34) (xy 181.61 38.1))
     (stroke (width 0) (type default))
   )
@@
     (stroke (width 0) (type default))
   )
-  (wire (pts (xy 190.5 72.39) (xy 190.5 81.28))
+  (wire (pts (xy 181.61 69.85) (xy 181.61 71.12))
     (stroke (width 0) (type default))
   )
@@
   )
   (wire (pts (xy 19.05 93.98) (xy 39.37 93.98))
-    (stroke (width 0) (type default))
-  )
-  (wire (pts (xy 190.5 55.88) (xy 190.5 64.77))
     (stroke (width 0) (type default))
   )
@@
     )
   )
-  (symbol (lib_id "power:GND") (at 190.5 95.25 0) (unit 1)
-    (in_bom yes) (on_board yes) (dnp no)
-    (property "Reference" "#PWR013" (at 190.5 101.6 0)
-      (effects (font (size 1.27 1.27)) hide)
-    )
-    (property "Value" "GND" (at 190.5 100.33 0)
-      (effects (font (size 1.27 1.27)))
-    )
-    (property "Footprint" "" (at 190.5 95.25 0)
-      (effects (font (size 1.27 1.27)) hide)
-    )
-    (property "Datasheet" "" (at 190.5 95.25 0)
+  (symbol (lib_id "power:GND") (at 181.61 82.55 0) (unit 1)
+    (in_bom yes) (on_board yes) (dnp no)
+    (property "Reference" "#PWR013" (at 181.61 88.9 0)
+      (effects (font (size 1.27 1.27)) hide)
+    )
+    (property "Value" "GND" (at 181.61 87.63 0)
+      (effects (font (size 1.27 1.27)))
+    )
+    (property "Footprint" "" (at 181.61 82.55 0)
+      (effects (font (size 1.27 1.27)) hide)
+    )
+    (property "Datasheet" "" (at 181.61 82.55 0)
       (effects (font (size 1.27 1.27)) hide)
     )
@@
     )
   )
-  (symbol (lib_id "Device:R_US") (at 181.61 53.34 90) (unit 1)
-    (in_bom yes) (on_board yes) (dnp no)
-    (property "Reference" "R1" (at 181.61 46.99 90)
-      (effects (font (size 1.27 1.27)))
-    )
-    (property "Value" "10K" (at 181.61 49.53 90)
-      (effects (font (size 1.27 1.27)))
-    )
-    (property "Footprint" "" (at 181.864 52.324 90)
-      (effects (font (size 1.27 1.27)) hide)
-    )
-    (property "Datasheet" "~" (at 181.61 53.34 0)
+  (symbol (lib_id "Device:R_US") (at 173.99 53.34 90) (unit 1)
+    (in_bom yes) (on_board yes) (dnp no)
+    (property "Reference" "R1" (at 173.99 46.99 90)
+      (effects (font (size 1.27 1.27)))
+    )
+    (property "Value" "10K" (at 173.99 49.53 90)
+      (effects (font (size 1.27 1.27)))
+    )
+    (property "Footprint" "" (at 174.244 52.324 90)
+      (effects (font (size 1.27 1.27)) hide)
+    )
+    (property "Datasheet" "~" (at 173.99 53.34 0)
       (effects (font (size 1.27 1.27)) hide)
     )
@@
     )
   )
-  (symbol (lib_id "power:+5P") (at 151.13 31.75 0) (unit 1)
+  (symbol (lib_id "power:+5P") (at 151.13 34.29 0) (unit 1)
     (in_bom yes) (on_board yes) (dnp no) (fields_autoplaced)
-    (property "Reference" "#PWR01" (at 151.13 35.56 0)
-      (effects (font (size 1.27 1.27)) hide)
-    )
-    (property "Value" "+5P" (at 151.13 26.67 0)
-      (effects (font (size 1.27 1.27)))
-    )
-    (property "Footprint" "" (at 151.13 31.75 0)
-      (effects (font (size 1.27 1.27)) hide)
-    )
-    (property "Datasheet" "" (at 151.13 31.75 0)
+    (property "Reference" "#PWR01" (at 151.13 38.1 0)
+      (effects (font (size 1.27 1.27)) hide)
+    )
+    (property "Value" "+5P" (at 151.13 29.21 0)
+      (effects (font (size 1.27 1.27)))
+    )
+    (property "Footprint" "" (at 151.13 34.29 0)
+      (effects (font (size 1.27 1.27)) hide)
+    )
+    (property "Datasheet" "" (at 151.13 34.29 0)
       (effects (font (size 1.27 1.27)) hide)
     )
@@
     )
   )
-  (symbol (lib_id "Device:LED") (at 190.5 85.09 90) (unit 1)
+  (symbol (lib_id "Device:LED") (at 181.61 74.93 90) (unit 1)
     (in_bom yes) (on_board yes) (dnp no) (fields_autoplaced)
-    (property "Reference" "D1" (at 194.31 85.4075 90)
-      (effects (font (size 1.27 1.27)) (justify right))
-    )
-    (property "Value" "LED" (at 194.31 87.9475 90)
-      (effects (font (size 1.27 1.27)) (justify right))
-    )
-    (property "Footprint" "" (at 190.5 85.09 0)
-      (effects (font (size 1.27 1.27)) hide)
-    )
-    (property "Datasheet" "~" (at 190.5 85.09 0)
+    (property "Reference" "D1" (at 185.42 75.2475 90)
+      (effects (font (size 1.27 1.27)) (justify right))
+    )
+    (property "Value" "LED" (at 185.42 77.7875 90)
+      (effects (font (size 1.27 1.27)) (justify right))
+    )
+    (property "Footprint" "" (at 181.61 74.93 0)
+      (effects (font (size 1.27 1.27)) hide)
+    )
+    (property "Datasheet" "~" (at 181.61 74.93 0)
       (effects (font (size 1.27 1.27)) hide)
     )
@@
     )
   )
-  (symbol (lib_id "Device:R_US") (at 190.5 68.58 0) (unit 1)
-    (in_bom yes) (on_board yes) (dnp no)
-    (property "Reference" "R3" (at 194.31 69.85 90)
-      (effects (font (size 1.27 1.27)))
-    )
-    (property "Value" "1K" (at 194.31 67.31 90)
-      (effects (font (size 1.27 1.27)))
-    )
-    (property "Footprint" "" (at 191.516 68.834 90)
-      (effects (font (size 1.27 1.27)) hide)
-    )
-    (property "Datasheet" "~" (at 190.5 68.58 0)
+  (symbol (lib_id "Device:R_US") (at 181.61 66.04 0) (unit 1)
+    (in_bom yes) (on_board yes) (dnp no)
+    (property "Reference" "R3" (at 185.42 67.31 90)
+      (effects (font (size 1.27 1.27)))
+    )
+    (property "Value" "1K" (at 185.42 64.77 90)
+      (effects (font (size 1.27 1.27)))
+    )
+    (property "Footprint" "" (at 182.626 66.294 90)
+      (effects (font (size 1.27 1.27)) hide)
+    )
+    (property "Datasheet" "~" (at 181.61 66.04 0)
       (effects (font (size 1.27 1.27)) hide)
     )
@@
     )
   )
-  (symbol (lib_id "power:GND") (at 151.13 76.2 0) (unit 1)
-    (in_bom yes) (on_board yes) (dnp no)
-    (property "Reference" "#PWR03" (at 151.13 82.55 0)
-      (effects (font (size 1.27 1.27)) hide)
-    )
-    (property "Value" "GND" (at 151.13 81.28 0)
-      (effects (font (size 1.27 1.27)))
-    )
-    (property "Footprint" "" (at 151.13 76.2 0)
-      (effects (font (size 1.27 1.27)) hide)
-    )
-    (property "Datasheet" "" (at 151.13 76.2 0)
-      (effects (font (size 1.27 1.27)) hide)
-    )
+  (symbol (lib_id "power:GND") (at 151.13 72.39 0) (unit 1)
+    (in_bom yes) (on_board yes) (dnp no)
+    (property "Reference" "#PWR03" (at 151.13 78.74 0)
+      (effects (font (size 1.27 1.27)) hide)
+    )
+    (property "Value" "GND" (at 151.13 77.47 0)
+      (effects (font (size 1.27 1.27)))
+    )
+    (property "Footprint" "" (at 151.13 72.39 0)
+      (effects (font (size 1.27 1.27)) hide)
+    )
+    (property "Datasheet" "" (at 151.13 72.39 0)
+      (effects (font (size 1.27 1.27)) hide)
+    )
