File: projects/21-I2C_WITH_PIC10F2XX/PIC10F222/KiCad/PIC10F222_I2C.kicad_sch (KiCad schematic)
At the start: 1 part, among them U1 PIC10F222-IP

Commit message: Doc
Parts:
- added R1, R2, R4: 4.7K, symbol Device:R
- added R3: 10K, symbol Device:R
- added SW1, SW2: SW_Push, symbol Switch:SW_Push
- added U2: RDA5807M, symbol RF_Module:RDA5807M
Connections:
- net +5V: now also R1.1, R2.1, R3.1, R4.1, U2.5 (VCC)
- net GND: now also U2.6 (GND)
- net at U1.3 (GP2): now also SW2.1
- net at U1.4 (GP1): now also R1.2, U2.2 (SCL)
- net at U1.5 (GP0): now also R2.2, U2.1 (SDA)
- net at U1.8 (GP3): now also SW1.1
- new net: R4.2, SW2.2
- new net: R3.2, SW1.2
